File: circuit/mini.brd (EAGLE design)
At the start: 100 x 80 mm, 80 parts, among them IC1 74AC4053D, IC2 74AC74D, IC3 STM32L151CBT6, IC4 MCP1700-3.3V, IC5 NE5534D, IC6 NE5534D, Q1 BFG135, Q2 8MHz, X1 1-227161-0, X4 MINI-USB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

Commit message: - ??????? ????????? ??? ????? ???????????? ??????????
Parts:
- moved C30 58.3 mm to (72.4, 21.0)
- moved R28 57.2 mm to (77.5, 22.9)
- moved R22 56.0 mm to (84.5, 27.9)
- moved R25 56.0 mm to (76.8, 29.2)
- moved R23 55.9 mm to (83.8, 22.9)
- moved C24 51.2 mm to (72.4, 66.0)
- moved C10 50.5 mm to (88.3, 31.8)
- moved R29 49.6 mm to (69.8, 31.1)
- moved C23 47.1 mm to (72.4, 69.8)
- moved R19 40.3 mm to (80.0, 61.6)
- moved C34 28.8 mm to (89.5, 47.0)
- moved R18 28.7 mm to (81.3, 64.8)
- moved R17 28.3 mm to (77.5, 64.8)
- moved C38 24.8 mm to (92.7, 43.2)
- moved IC6 22.4 mm to (81.9, 42.5)
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
Commit message: - ????????? ??????????? AD9850 ??????
Parts:
- removed X5: SWD, con-cypressindustries:32005-301
- added C31: 100n, rcl:C0603
- added X6: (no value), con-phoenix-254:4POL254
- moved R6 23.9 mm to (56.5, 34.9)
- moved R7 17.8 mm to (52.7, 34.9), turned to 180 degrees
- moved X2 13.0 mm to (50.2, 30.5), turned to 180 degrees
- moved X3 13.0 mm to (50.2, 10.0), turned to 180 degrees
- moved IC2 10.8 mm to (50.2, 44.5)
Connections:
- net +3V3: now also X6.1; no longer X5.1
- net +5V: now also C31.1
- net AD7: now also IC3.40; no longer IC3.41
- net A_RESET: now also IC3.39; no longer IC3.42
- net FQ_UD: now also IC3.41; no longer IC3.40
- net GND: now also C31.2, X6.4; no longer X5.5, X5.M1, X5.M2, X5.M3, X5.M4
- net SWDCLK: now also X6.3; no longer X5.3
- net SWDIO: now also X6.2; no longer X5.2
- net W_CLK: now also IC3.42; no longer IC3.39
Routing:
- net N$31: track 55.5 -> 10.7 mm, vias 2 -> 0
- net +5V: track 52.8 -> 91.3 mm, vias 0 -> 2
- net GND: track 318.0 -> 339.4 mm, vias 0 -> 2
- net W_CLK: track 37.9 -> 22.2 mm
- net +3V3: track 37.3 -> 50.0 mm, vias 0 -> 2
- net VCC: track 86.3 -> 75.6 mm, vias 2 -> 4
- net FQ_UD: track 34.8 -> 26.1 mm
- net N$2: track 20.8 -> 28.5 mm
- net SWDCLK: track 12.9 -> 17.4 mm
- net N$1: track 26.3 -> 22.2 mm
- net A_RESET: track 28.6 -> 32.3 mm
- net SWDIO: track 10.8 -> 14.6 mm
- net N$4: track 7.66 -> 10.3 mm
- net AD7: track 31.7 -> 29.2 mm
- net N$32: track 20.1 -> 22.4 mm
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
Commit message: - ??????? ?????? ?????????
Parts:
- removed C10: 100n, rcl:C0603
- added C32: 1mk, rcl:C0603
- added X5: (no value), con-phoenix-254:4POL254
- moved R29 43.4 mm to (81.3, 73.0)
- moved R20 36.0 mm to (70.5, 40.6)
- moved R23 34.7 mm to (69.8, 54.6)
- moved C30 31.2 mm to (69.8, 52.1), turned to 180 degrees
- moved R28 31.2 mm to (80.0, 54.0)
- moved R21 31.0 mm to (70.5, 48.9)
- moved C22 30.7 mm to (69.2, 46.4)
- moved R22 28.5 mm to (74.3, 54.6)
- moved C21 28.4 mm to (69.2, 43.2)
- moved R25 23.0 mm to (74.3, 52.1)
- moved C19 19.1 mm to (64.8, 40.6), turned to 180 degrees
- moved R19 16.4 mm to (70.5, 74.9)
- moved R14 15.9 mm to (64.8, 43.2)
- moved R24 13.9 mm to (74.3, 71.8)
- moved C38 12.9 mm to (85.7, 54.0)
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Connections:
- new net N$38: C37.2, X5.1
- new net N$39: C38.2, X5.3
- net +5V: now also C32.1; no longer C10.1
- net GND: now also C32.2, X5.2, X5.4; no longer C10.2
Routing:
- net GND: track 339.4 -> 552.9 mm, vias 2 -> 10
- net +5V: track 91.3 -> 217.7 mm, vias 2 -> 6
- net N$5: track 0.00 -> 34.4 mm, vias 0 -> 2
- net N$8: track 0.00 -> 28.3 mm, vias 0 -> 2
- net N$16: track 0.00 -> 23.0 mm
- net N$39: track 0.00 -> 20.6 mm
- net N$10: track 0.00 -> 20.5 mm, vias 0 -> 2
- net N$22: track 0.00 -> 19.4 mm
- net N$17: track 0.00 -> 19.1 mm
- net N$18: track 0.00 -> 18.6 mm
- net N$9: track 0.00 -> 17.1 mm, vias 0 -> 2
- net N$26: track 0.00 -> 14.1 mm
- net N$24: track 0.00 -> 12.2 mm
- net N$38: track 0.00 -> 10.1 mm
- net N$23: track 0.00 -> 7.82 mm
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
Commit message: - ?????? ???????????
Parts:
- moved C14 19.8 mm to (59.7, 59.7)
Routing:
- net GND: track 552.9 -> 542.0 mm
- net +5V: track 217.7 -> 216.4 mm
Changed lines of the file:
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@@
 <element name="L2" library="rcl" package="L3225M" value="470nH" x="21.59" y="62.23"/>
 <element name="C6" library="rcl" package="C0603" value="100n" x="26.67" y="58.42"/>
-<element name="C14" library="rcl" package="C0603" value="100n" x="45.085" y="73.025" rot="R180"/>
+<element name="C14" library="rcl" package="C0603" value="100n" x="59.69" y="59.69" rot="R180"/>
 <element name="X1" library="con-coax" package="AMP_227161" value="1-227161-0" x="7.62" y="55.88" rot="R90">
 <attribute name="OC_NEWARK" value="33B3200" x="17.78" y="78.74" size="1.778" layer="27" rot="R90" display="off"/>
@@
 <wire x1="47.0916" y1="40.64" x2="50.8" y2="40.64" width="0.6096" layer="1"/>
 <wire x1="47.0916" y1="40.64" x2="47.0916" y2="41.91" width="0.6096" layer="1"/>
-<wire x1="45.935" y1="73.025" x2="45.935" y2="71.54" width="0.4064" layer="1"/>
-<wire x1="45.935" y1="71.54" x2="46.355" y2="71.12" width="0.4064" layer="1"/>
 <wire x1="7.305" y1="27.305" x2="7.305" y2="29.745" width="0.4064" layer="1"/>
 <wire x1="7.305" y1="29.745" x2="7.405" y2="29.845" width="0.4064" layer="1"/>
@@
 <wire x1="53.2384" y1="44.45" x2="59.055" y2="44.45" width="0.4064" layer="1"/>
 <wire x1="59.055" y1="44.45" x2="60.325" y2="45.72" width="0.4064" layer="1"/>
-<wire x1="60.325" y1="45.72" x2="60.325" y2="64.135" width="0.4064" layer="1"/>
+<wire x1="60.325" y1="45.72" x2="60.325" y2="60.325" width="0.4064" layer="1"/>
+<wire x1="60.325" y1="60.325" x2="60.325" y2="64.135" width="0.4064" layer="1"/>
 <wire x1="60.325" y1="64.135" x2="58.42" y2="66.04" width="0.4064" layer="1"/>
 <wire x1="58.42" y1="66.04" x2="56.4134" y2="66.04" width="0.4064" layer="1"/>
@@
 <via x="77.47" y="56.515" extent="1-16" drill="0.6" diameter="1.4224" shape="square"/>
 <wire x1="77.47" y1="56.515" x2="77.47" y2="59.055" width="0.4064" layer="1"/>
+<wire x1="60.54" y1="59.69" x2="60.54" y2="60.11" width="0.4064" layer="1"/>
+<wire x1="60.54" y1="60.11" x2="60.325" y2="60.325" width="0.4064" layer="1"/>
 </signal>
 <signal name="GND">
@@
 <wire x1="14.605" y1="34.925" x2="14.605" y2="32.49925625" width="0.4064" layer="1"/>
 <wire x1="14.605" y1="32.49925625" x2="15.742225" y2="31.36203125" width="0.4064" layer="1"/>
-<wire x1="44.235" y1="73.025" x2="36.195" y2="73.025" width="0.4064" layer="1"/>
-<wire x1="36.195" y1="73.025" x2="33.655" y2="70.485" width="0.4064" layer="1"/>
-<wire x1="33.655" y1="70.485" x2="33.655" y2="68.795" width="0.4064" layer="1"/>
 <wire x1="33.655" y1="68.795" x2="33.44" y2="68.58" width="0.4064" layer="1"/>
 <wire x1="8.04" y1="14.605" x2="8.04" y2="11.365" width="0.4064" layer="1"/>
@@
 <wire x1="10.795" y1="46.355" x2="2.54" y2="38.1" width="0.4064" layer="1"/>
 <wire x1="2.54" y1="38.1" x2="2.54" y2="25.4" width="0.4064" layer="1"/>
+<wire x1="10.795" y1="53.34" x2="10.16" y2="53.975" width="0.4064" layer="1"/>
+<wire x1="58.84" y1="59.69" x2="56.4134" y2="59.69" width="0.4064" layer="1"/>
 <wire x1="97.155" y1="62.23" x2="99.06" y2="62.23" width="0" layer="19" extent="1-1"/>
 <wire x1="9.105" y1="29.845" x2="9.205" y2="27.305" width="0" layer="19" extent="1-1"/>
-<wire x1="10.795" y1="53.34" x2="10.16" y2="53.975" width="0.4064" layer="1"/>
 </signal>
 <signal name="N$1">

Commit message: - ?????? ???? ?????? ??????? ????? ??
Parts:
- removed C29, C30: 1mk, rcl:C0603
- removed R24, R25: 10K, rcl:R0603
- R18, R19, R22, R23: value 10K -> 22K
- moved R23 4.96 mm to (73.0, 50.8)
- moved R22 4.26 mm to (76.2, 50.8)
- moved R19 3.70 mm to (72.4, 71.8)
- moved R20 3.59 mm to (73.0, 43.2)
- moved R18 3.42 mm to (75.6, 71.8)
- moved R16 3.18 mm to (72.4, 63.5)
- moved R21 2.84 mm to (73.0, 47.6)
- moved R17 2.01 mm to (72.4, 68.6)
- moved C8 1.80 mm to (35.6, 67.3), turned to 270 degrees
Connections:
- removed net N$24: IC6.3, R21.2, R25.2
- removed net N$26: IC5.3, R17.2, R24.2
- net GND: no longer C29.2, C30.2
- net N$15: now also IC5.3, R17.2; no longer C29.1, R24.1
- net N$23: now also IC6.3, R21.2; no longer C30.1, R25.1
Routing:
- net GND: track 542.0 -> 500.8 mm, vias 10 -> 8
- net N$26: track 14.1 -> 0.00 mm
- net N$24: track 12.2 -> 0.00 mm
- net N$15: track 7.40 -> 12.6 mm
- net +5V: track 216.4 -> 221.4 mm
- net N$22: track 19.4 -> 15.7 mm
- net N$17: track 19.1 -> 15.7 mm
- net N$23: track 7.82 -> 10.9 mm
- net N$21: track 0.00 -> 2.64 mm
- net N$37: track 5.77 -> 4.74 mm
- net N$20: track 2.72 -> 2.11 mm
- net N$19: track 2.62 -> 2.11 mm

Commit message: - ??? ??????????????????. - ???????? ??????, ????? ???????? ????????????? ??????? ????????.
Parts:
- added X7: (no value), con-phoenix-254:2POL254
- moved X4 80.7 mm to (91.4, 26.0), turned to 180 degrees
- moved C26 76.6 mm to (85.1, 22.2), turned to 270 degrees
- moved X6 74.1 mm to (92.7, 39.4), turned to 90 degrees
- moved IC4 71.8 mm to (80.0, 21.6), turned to 270 degrees
- moved L3 70.8 mm to (74.9, 17.8), turned to 0 degrees
- moved R27 70.3 mm to (85.1, 29.8), turned to 270 degrees
- moved C33 68.0 mm to (76.2, 21.6), turned to 90 degrees
- moved C12 67.5 mm to (79.4, 25.4), turned to 0 degrees
- moved R26 67.3 mm to (82.5, 29.8), turned to 270 degrees
- moved C16 64.4 mm to (72.4, 21.6), turned to 90 degrees
- moved C11 62.3 mm to (81.9, 35.6), turned to 90 degrees
- moved C15 62.1 mm to (69.8, 21.6), turned to 90 degrees
- moved IC3 57.7 mm to (75.6, 31.8), turned to 270 degrees
- moved C25 51.8 mm to (68.3, 29.1), turned to 270 degrees
- moved C28 49.6 mm to (66.0, 31.8), turned to 180 degrees
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Connections:
- net AD7: now also IC3.14; no longer IC3.40
- net A_RESET: now also IC3.13; no longer IC3.39
- net FQ_UD: now also IC3.15; no longer IC3.41
- net I-LO: now also X7.1
- net Q-LO: now also X7.2
- net W_CLK: now also IC3.16; no longer IC3.42
Routing:
- net GND: track 500.8 -> 404.8 mm, vias 8 -> 6
- net +5V: track 221.4 -> 185.3 mm, vias 6 -> 8
- net W_CLK: track 22.2 -> 43.9 mm
- net N$32: track 22.4 -> 2.69 mm
- net FQ_UD: track 26.1 -> 40.2 mm
- net N$39: track 20.6 -> 7.57 mm
- net QOUT: track 4.60 -> 16.6 mm
- net VCC: track 75.6 -> 83.4 mm, vias 4 -> 2
- net N$2: track 28.5 -> 22.1 mm
- net AD7: track 29.2 -> 35.5 mm
- net N$5: track 34.4 -> 28.0 mm
- net N$16: track 23.0 -> 16.9 mm
- net N$38: track 10.1 -> 3.94 mm
- net N$31: track 10.7 -> 4.72 mm
- net N$3: track 13.3 -> 7.51 mm
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
Commit message: - ?????????????????? ?? ??????? 85x60??
Parts:
- moved C32 25.7 mm to (59.7, 47.6), turned to 180 degrees
- moved C1 22.2 mm to (16.5, 32.4)
- moved C2 22.2 mm to (17.1, 36.2)
- moved C3 22.2 mm to (19.7, 32.4)
- moved X1 22.2 mm to (7.62, 33.7)
- moved L1 22.2 mm to (13.3, 40.0)
- moved R29 21.6 mm to (72.4, 53.3), turned to 270 degrees
- moved R18 21.1 mm to (59.7, 57.8), turned to 90 degrees
- moved C36 20.3 mm to (70.5, 53.3), turned to 270 degrees
- moved R19 19.9 mm to (62.2, 54.6), turned to 90 degrees
- moved X5 19.8 mm to (76.2, 50.2)
- moved R17 19.3 mm to (59.1, 54.6)
- moved R28 19.0 mm to (73.0, 40.0), turned to 270 degrees
- moved C38 18.9 mm to (73.0, 44.5)
- moved C24 18.4 mm to (55.9, 53.3)
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Routing:
- net GND: track 404.8 -> 397.9 mm
- net N$18: track 18.4 -> 12.6 mm
- net +5V: track 185.3 -> 180.4 mm
- net N$17: track 15.7 -> 19.6 mm
- net N$22: track 13.2 -> 16.8 mm
- net N$41: track 19.2 -> 21.9 mm
- net N$44: track 12.1 -> 9.53 mm
- net N$13: track 4.69 -> 6.26 mm
- net N$39: track 7.57 -> 6.30 mm
- net N$6: track 20.3 -> 19.0 mm
- net N$21: track 2.64 -> 3.68 mm
- net N$25: track 2.90 -> 2.00 mm
- net N$16: track 16.9 -> 17.7 mm
- net N$34: track 19.6 -> 18.8 mm
- net N$38: track 3.94 -> 3.20 mm
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Other:
- board size 100 x 80 mm -> 84.8 x 61 mm

Commit message: - ???????? ????? ??????? ? ????????? ???????? 78x61 ??
Parts:
- moved C2 16.6 mm to (5.71, 48.3), turned to 90 degrees
- moved C3 13.7 mm to (6.99, 37.5)
- moved C6 9.52 mm to (11.4, 52.7)
- moved L1 9.38 mm to (8.89, 48.3)
- moved C4 9.03 mm to (7.62, 52.7)
- moved L2 8.64 mm to (9.53, 56.5)
- moved C1 8.13 mm to (10.2, 37.5)
- moved C11 5.72 mm to (63.5, 24.1)
- moved C13 5.72 mm to (52.7, 26.0)
- moved C18 5.72 mm to (46.4, 57.1)
- moved C20 5.72 mm to (46.4, 49.5)
- moved C21 5.72 mm to (50.8, 37.5)
- moved C22 5.72 mm to (50.8, 40.0)
- moved C23 5.72 mm to (50.2, 50.8)
- moved C24 5.72 mm to (50.2, 53.3)
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Routing:
- net N$41: track 21.9 -> 29.3 mm
- net GND: track 397.9 -> 392.8 mm, vias 6 -> 10
- net N$40: track 12.3 -> 15.3 mm
- net N$33: track 10.1 -> 12.2 mm
- net N$44: track 9.53 -> 10.6 mm
- net N$5: track 28.2 -> 29.2 mm
- net +5V: track 180.4 -> 179.9 mm
- added copper zone on layer 1, net GND
Other:
- board size 84.8 x 61 mm -> 77.8 x 61 mm
- board text added: "BALMER"
- board text added: "SDR 2014"
