File: circuit/mini.brd (EAGLE design)
At the start: 77.8 x 61 mm, 79 parts, among them IC1 74AC4053D, IC2 74AC74D, IC3 STM32L151CBT6, IC4 MCP1700-3.3V, IC5 NE5534D, IC6 NE5534D, Q1 BFG135, Q2 8MHz, X1 1-227161-0, X4 MINI-USB

Commit message: - ????? ??? USB ?????
Routing:
- net GND: vias 10 -> 12

Commit message: - ?????????? USB ? ????????? ??????? ??? AD9850
Parts:
- R2, R8, R9: value 1K -> 1K5
- moved C3 15.5 mm to (4.45, 52.7), turned to 90 degrees
- moved C1 6.48 mm to (16.5, 38.7), turned to 90 degrees
- flipped X1 to the bottom, turned to 270 degrees
Routing:
- net GND: track 392.8 -> 454.2 mm
- net N$41: track 29.3 -> 15.2 mm
- net N$18: track 12.6 -> 8.94 mm
- net N$40: track 15.3 -> 18.6 mm

Commit message: - ????????? ????? - ?????????? ?????????? ?????? ??? IC5
Connections:
- net N$10: now also IC1.1; no longer IC1.2
- net N$9: now also IC1.2; no longer IC1.1
Routing:
- net GND: track 454.2 -> 479.2 mm
- net N$18: track 8.94 -> 14.5 mm
- net N$9: track 17.4 -> 20.7 mm
- net N$10: track 20.5 -> 22.9 mm
Changed lines of the file:
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@@
 <wire x1="76.025" y1="10.155" x2="76.025" y2="4.905" width="0.4064" layer="1"/>
 <wire x1="76.025" y1="4.905" x2="74.295" y2="3.175" width="0.4064" layer="1"/>
-<wire x1="26.035" y1="3.65" x2="3.65" y2="3.65" width="0" layer="19" extent="1-16"/>
-<wire x1="3.65" y1="3.65" x2="3.175" y2="3.175" width="0.4064" layer="1"/>
 <wire x1="2.855" y1="53.655" x2="2.855" y2="57.465" width="0.4064" layer="1"/>
 <wire x1="2.855" y1="57.465" x2="3.175" y2="57.785" width="0.4064" layer="1"/>
+<wire x1="26.035" y1="3.65" x2="26.035" y2="1.905" width="0.4064" layer="1"/>
+<wire x1="26.035" y1="1.905" x2="25.4" y2="1.27" width="0.4064" layer="1"/>
+<wire x1="25.4" y1="1.27" x2="5.08" y2="1.27" width="0.4064" layer="1"/>
+<wire x1="5.08" y1="1.27" x2="3.175" y2="3.175" width="0.4064" layer="1"/>
 </signal>
 <signal name="N$1">
@@
 <wire x1="31.8516" y1="49.53" x2="29.845" y2="49.53" width="0.4064" layer="1"/>
 <wire x1="29.845" y1="49.53" x2="29.21" y2="48.895" width="0.4064" layer="1"/>
-</signal>
-<signal name="N$9">
-<contactref element="IC1" pad="1"/>
-<contactref element="R13" pad="1"/>
-<via x="43.18" y="55.245" extent="1-16" drill="0.6" diameter="1.4224" shape="square"/>
-<wire x1="43.18" y1="55.245" x2="32.385" y2="55.245" width="0.4064" layer="16"/>
-<wire x1="32.385" y1="55.245" x2="31.115" y2="56.515" width="0.4064" layer="16"/>
-<via x="31.115" y="56.515" extent="1-16" drill="0.6" diameter="1.4224" shape="square"/>
-<wire x1="31.115" y1="56.515" x2="31.115" y2="55.3466" width="0.4064" layer="1"/>
-<wire x1="31.115" y1="55.3466" x2="31.8516" y2="54.61" width="0.4064" layer="1"/>
-<wire x1="43.18" y1="55.245" x2="44.87" y2="55.245" width="0.4064" layer="1"/>
-<wire x1="44.87" y1="55.245" x2="45.505" y2="54.61" width="0.4064" layer="1"/>
-</signal>
-<signal name="N$10">
-<contactref element="IC1" pad="2"/>
-<contactref element="R12" pad="1"/>
-<wire x1="45.505" y1="52.07" x2="43.18" y2="52.07" width="0.4064" layer="1"/>
-<via x="43.18" y="52.07" extent="1-16" drill="0.6" diameter="1.4224" shape="square"/>
-<wire x1="43.18" y1="52.07" x2="31.75" y2="52.07" width="0.4064" layer="16"/>
-<wire x1="31.75" y1="52.07" x2="29.21" y2="54.61" width="0.4064" layer="16"/>
-<via x="29.21" y="54.61" extent="1-16" drill="0.6" diameter="1.4224" shape="square"/>
-<wire x1="29.21" y1="54.61" x2="30.48" y2="53.34" width="0.4064" layer="1"/>
-<wire x1="30.48" y1="53.34" x2="31.8516" y2="53.34" width="0.4064" layer="1"/>
 </signal>
 <signal name="N$11">
@@
 <wire x1="64.77" y1="52.39" x2="66.575" y2="52.39" width="0.4064" layer="1"/>
 <wire x1="66.575" y1="52.39" x2="66.675" y2="52.49" width="0.4064" layer="1"/>
-<wire x1="66.675" y1="52.49" x2="66.675" y2="56.195" width="0" layer="19" extent="1-16"/>
 <wire x1="66.675" y1="56.195" x2="66.995" y2="56.515" width="0.4064" layer="1"/>
+<wire x1="66.675" y1="52.49" x2="67.73" y2="52.49" width="0.4064" layer="1"/>
+<wire x1="67.73" y1="52.49" x2="67.945" y2="52.705" width="0.4064" layer="1"/>
+<wire x1="67.945" y1="52.705" x2="67.945" y2="55.245" width="0.4064" layer="1"/>
+<wire x1="67.945" y1="55.245" x2="67.31" y2="55.88" width="0.4064" layer="1"/>
+<wire x1="67.31" y1="55.88" x2="67.31" y2="56.2" width="0.4064" layer="1"/>
+<wire x1="67.31" y1="56.2" x2="66.995" y2="56.515" width="0.4064" layer="1"/>
 </signal>
 <signal name="N$20">
@@
 <wire x1="69.85" y1="48.26" x2="70.485" y2="48.895" width="0.4064" layer="1"/>
 </signal>
+<signal name="N$9">
+<contactref element="IC1" pad="2"/>
+<contactref element="R13" pad="1"/>
+<wire x1="45.505" y1="54.61" x2="43.815" y2="54.61" width="0.4064" layer="1"/>
+<via x="43.815" y="54.61" extent="1-16" drill="0.6" diameter="1.4224" shape="square"/>
+<wire x1="43.815" y1="54.61" x2="28.575" y2="54.61" width="0.4064" layer="16"/>
+<via x="28.575" y="54.61" extent="1-16" drill="0.6" diameter="1.4224" shape="square"/>
+<wire x1="28.575" y1="54.61" x2="29.21" y2="54.61" width="0.4064" layer="1"/>
+<wire x1="29.21" y1="54.61" x2="29.845" y2="53.975" width="0.4064" layer="1"/>
+<wire x1="31.8516" y1="53.34" x2="30.48" y2="53.34" width="0.4064" layer="1"/>
+<wire x1="30.48" y1="53.34" x2="29.845" y2="53.975" width="0.4064" layer="1"/>
+</signal>
+<signal name="N$10">
+<contactref element="R12" pad="1"/>
+<contactref element="IC1" pad="1"/>
+<wire x1="31.8516" y1="54.61" x2="31.8516" y2="55.9816" width="0.4064" layer="1"/>
+<wire x1="31.8516" y1="55.9816" x2="32.385" y2="56.515" width="0.4064" layer="1"/>
+<via x="32.385" y="56.515" extent="1-16" drill="0.6" diameter="1.4224" shape="square"/>
+<wire x1="32.385" y1="56.515" x2="45.085" y2="56.515" width="0.4064" layer="16"/>
+<wire x1="45.085" y1="56.515" x2="46.355" y2="55.245" width="0.4064" layer="16"/>
+<wire x1="46.355" y1="55.245" x2="46.355" y2="53.975" width="0.4064" layer="16"/>
+<wire x1="46.355" y1="53.975" x2="44.45" y2="52.07" width="0.4064" layer="16"/>
+<wire x1="44.45" y1="52.07" x2="43.815" y2="52.07" width="0.4064" layer="16"/>
+<via x="43.815" y="52.07" extent="1-16" drill="0.6" diameter="1.4224" shape="square"/>
+<wire x1="43.815" y1="52.07" x2="45.505" y2="52.07" width="0.4064" layer="1"/>
+</signal>
 </signals>
