File: circuit/mini.sch (EAGLE design)
At the start: 83 parts, among them IC1 74AC4053D, IC2 74AC74D, IC3 STM32L151CBT6, IC4 MCP1700-3.3V, IC5 NE5534D, IC6 NE5534D, Q1 BFG135, Q2 8MHz, X1 B35N57, X4 MINI-USB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

Commit message: - enable serial mode
Connections:
- removed net AD0: X3-2.1
- removed net AD1: X3-3.1
- removed net AD2: X3-4.1
- net GND: now also X3-4.1
- net VCC: now also X3-2.1, X3-3.1
Other:
- note added: "AD0"
- note added: "AD1"
- note added: "AD2"
Changed lines of the file:
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@@
 <part name="C14" library="rcl" deviceset="C-EU" device="C0603" value="100n"/>
 <part name="X1" library="con-coax" deviceset="B35N57" device=""/>
+<part name="GND23" library="supply1" deviceset="GND" device=""/>
 </parts>
 <sheets>
@@
 <plain>
 <text x="-58.42" y="78.74" size="1.778" layer="91">18 Mhz filter</text>
+<text x="-35.306" y="23.368" size="1.778" layer="95">AD0</text>
+<text x="-35.306" y="18.288" size="1.778" layer="95">AD1</text>
+<text x="-35.306" y="13.208" size="1.778" layer="95">AD2</text>
 </plain>
 <instances>
@@
 <instance part="C14" gate="G$1" x="101.6" y="-7.62"/>
 <instance part="X1" gate="G$1" x="-83.82" y="55.88"/>
+<instance part="GND23" gate="1" x="-40.64" y="10.16"/>
 </instances>
 <busses>
@@
 <junction x="-17.78" y="48.26"/>
 </segment>
+<segment>
+<pinref part="X3" gate="-4" pin="1"/>
+<wire x1="-30.48" y1="12.7" x2="-35.56" y2="12.7" width="0.1524" layer="91"/>
+<pinref part="GND23" gate="1" pin="GND"/>
+<wire x1="-35.56" y1="12.7" x2="-40.64" y2="12.7" width="0.1524" layer="91"/>
+</segment>
 </net>
 <net name="N$1" class="0">
@@
 <wire x1="-33.02" y1="27.94" x2="-33.02" y2="30.48" width="0.1524" layer="91"/>
 <pinref part="P+11" gate="VCC" pin="VCC"/>
+<pinref part="X3" gate="-3" pin="1"/>
+<wire x1="-30.48" y1="17.78" x2="-35.56" y2="17.78" width="0.1524" layer="91"/>
+<pinref part="X3" gate="-2" pin="1"/>
+<wire x1="-30.48" y1="22.86" x2="-35.56" y2="22.86" width="0.1524" layer="91"/>
+<wire x1="-35.56" y1="17.78" x2="-35.56" y2="22.86" width="0.1524" layer="91"/>
+<wire x1="-35.56" y1="22.86" x2="-35.56" y2="27.94" width="0.1524" layer="91"/>
+<wire x1="-35.56" y1="27.94" x2="-33.02" y2="27.94" width="0.1524" layer="91"/>
+<junction x="-33.02" y="27.94"/>
 </segment>
 <segment>
@@
 </segment>
 </net>
-<net name="AD0" class="0">
-<segment>
-<pinref part="X3" gate="-2" pin="1"/>
-<wire x1="-30.48" y1="22.86" x2="-35.56" y2="22.86" width="0.1524" layer="91"/>
-<label x="-35.306" y="23.368" size="1.778" layer="95"/>
-</segment>
-</net>
-<net name="AD1" class="0">
-<segment>
-<pinref part="X3" gate="-3" pin="1"/>
-<wire x1="-30.48" y1="17.78" x2="-35.56" y2="17.78" width="0.1524" layer="91"/>
-<label x="-35.306" y="18.288" size="1.778" layer="95"/>
-</segment>
-</net>
-<net name="AD2" class="0">
-<segment>
-<pinref part="X3" gate="-4" pin="1"/>
-<wire x1="-30.48" y1="12.7" x2="-35.56" y2="12.7" width="0.1524" layer="91"/>
-<label x="-35.306" y="13.208" size="1.778" layer="95"/>
-</segment>
-</net>

Commit message: - change connector
Parts:
- X1: value B35N57 -> 1-227161-0; device con-coax:B35N57 -> con-coax:1-227161-0
Connections:
- removed net AD3: X3-5.1
- removed net AD4: X3-6.1
- removed net AD5: X3-7.1
- removed net AD6: X3-8.1
- new net N$36: X3-9.1
- net AD7: now also IC3PORTA_L.PA5; no longer X3-9.1
- net A_RESET: now also IC3PORTA_L.PA6
- net FQ_UD: now also IC3PORTA_L.PA4
- net GND: now also X3-5.1, X3-6.1, X3-7.1, X3-8.1
- net W_CLK: now also IC3PORTA_L.PA3
Other:
- note added: "AD3"
- note added: "AD4"
- note added: "AD5"
- note added: "AD6"
- note added: "AD7"
Changed lines of the file:
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@@
 <part name="C6" library="rcl" deviceset="C-EU" device="C0603" value="100n"/>
 <part name="C14" library="rcl" deviceset="C-EU" device="C0603" value="100n"/>
-<part name="X1" library="con-coax" deviceset="B35N57" device=""/>
 <part name="GND23" library="supply1" deviceset="GND" device=""/>
+<part name="X1" library="con-coax" deviceset="?227161*" device="1-" technology="-0"/>
 </parts>
 <sheets>
@@
 <text x="-35.306" y="18.288" size="1.778" layer="95">AD1</text>
 <text x="-35.306" y="13.208" size="1.778" layer="95">AD2</text>
+<text x="-35.306" y="8.128" size="1.778" layer="95">AD3</text>
+<text x="-35.306" y="3.302" size="1.778" layer="95">AD4</text>
+<text x="-35.306" y="-2.032" size="1.778" layer="95">AD5</text>
+<text x="-35.306" y="-6.858" size="1.778" layer="95">AD6</text>
+<text x="-35.56" y="-11.938" size="1.778" layer="95">AD7</text>
 </plain>
 <instances>
@@
 <instance part="X3" gate="-10" x="-27.94" y="-17.78"/>
 <instance part="GND19" gate="1" x="-33.02" y="-22.86"/>
-<instance part="P+11" gate="VCC" x="-33.02" y="33.02"/>
+<instance part="P+11" gate="VCC" x="-35.56" y="33.02"/>
 <instance part="P+12" gate="VCC" x="-73.66" y="33.02"/>
 <instance part="GND20" gate="1" x="-73.66" y="0"/>
@@
 <instance part="C6" gate="G$1" x="-30.48" y="58.42" rot="R90"/>
 <instance part="C14" gate="G$1" x="101.6" y="-7.62"/>
+<instance part="GND23" gate="1" x="-40.64" y="10.16"/>
 <instance part="X1" gate="G$1" x="-83.82" y="55.88"/>
-<instance part="GND23" gate="1" x="-40.64" y="10.16"/>
 </instances>
 <busses>
@@
 <wire x1="-55.88" y1="48.26" x2="-38.1" y2="48.26" width="0.1524" layer="91"/>
 <wire x1="-38.1" y1="48.26" x2="-17.78" y2="48.26" width="0.1524" layer="91"/>
-<pinref part="X1" gate="G$1" pin="2"/>
 <wire x1="-71.12" y1="48.26" x2="-81.28" y2="48.26" width="0.1524" layer="91"/>
 <wire x1="-81.28" y1="48.26" x2="-81.28" y2="53.34" width="0.1524" layer="91"/>
@@
 <junction x="-38.1" y="48.26"/>
 <junction x="-17.78" y="48.26"/>
+<pinref part="X1" gate="G$1" pin="2"/>
 </segment>
 <segment>
@@
 <pinref part="GND23" gate="1" pin="GND"/>
 <wire x1="-35.56" y1="12.7" x2="-40.64" y2="12.7" width="0.1524" layer="91"/>
+<pinref part="X3" gate="-5" pin="1"/>
+<wire x1="-30.48" y1="7.62" x2="-35.56" y2="7.62" width="0.1524" layer="91"/>
+<wire x1="-35.56" y1="12.7" x2="-35.56" y2="7.62" width="0.1524" layer="91"/>
+<pinref part="X3" gate="-6" pin="1"/>
+<wire x1="-30.48" y1="2.54" x2="-35.56" y2="2.54" width="0.1524" layer="91"/>
+<wire x1="-35.56" y1="7.62" x2="-35.56" y2="2.54" width="0.1524" layer="91"/>
+<pinref part="X3" gate="-7" pin="1"/>
+<wire x1="-30.48" y1="-2.54" x2="-35.56" y2="-2.54" width="0.1524" layer="91"/>
+<wire x1="-35.56" y1="2.54" x2="-35.56" y2="-2.54" width="0.1524" layer="91"/>
+<pinref part="X3" gate="-8" pin="1"/>
+<wire x1="-30.48" y1="-7.62" x2="-35.56" y2="-7.62" width="0.1524" layer="91"/>
+<wire x1="-35.56" y1="-2.54" x2="-35.56" y2="-7.62" width="0.1524" layer="91"/>
+<junction x="-35.56" y="-2.54"/>
+<junction x="-35.56" y="2.54"/>
+<junction x="-35.56" y="7.62"/>
+<junction x="-35.56" y="12.7"/>
 </segment>
 </net>
@@
 </segment>
 <segment>
+<pinref part="X2" gate="-1" pin="1"/>
+<wire x1="-71.12" y1="27.94" x2="-73.66" y2="27.94" width="0.1524" layer="91"/>
+<wire x1="-73.66" y1="27.94" x2="-73.66" y2="30.48" width="0.1524" layer="91"/>
+<pinref part="P+12" gate="VCC" pin="VCC"/>
+</segment>
+<segment>
 <pinref part="X3" gate="-1" pin="1"/>
-<wire x1="-30.48" y1="27.94" x2="-33.02" y2="27.94" width="0.1524" layer="91"/>
-<wire x1="-33.02" y1="27.94" x2="-33.02" y2="30.48" width="0.1524" layer="91"/>
-<pinref part="P+11" gate="VCC" pin="VCC"/>
 <pinref part="X3" gate="-3" pin="1"/>
 <wire x1="-30.48" y1="17.78" x2="-35.56" y2="17.78" width="0.1524" layer="91"/>
@@
 <wire x1="-35.56" y1="17.78" x2="-35.56" y2="22.86" width="0.1524" layer="91"/>
 <wire x1="-35.56" y1="22.86" x2="-35.56" y2="27.94" width="0.1524" layer="91"/>
-<wire x1="-35.56" y1="27.94" x2="-33.02" y2="27.94" width="0.1524" layer="91"/>
-<junction x="-33.02" y="27.94"/>
-</segment>
-<segment>
-<pinref part="X2" gate="-1" pin="1"/>
-<wire x1="-71.12" y1="27.94" x2="-73.66" y2="27.94" width="0.1524" layer="91"/>
-<wire x1="-73.66" y1="27.94" x2="-73.66" y2="30.48" width="0.1524" layer="91"/>
-<pinref part="P+12" gate="VCC" pin="VCC"/>
+<wire x1="-35.56" y1="27.94" x2="-30.48" y2="27.94" width="0.1524" layer="91"/>
+<junction x="-35.56" y="22.86"/>
+<pinref part="P+11" gate="VCC" pin="VCC"/>
+<wire x1="-35.56" y1="30.48" x2="-35.56" y2="27.94" width="0.1524" layer="91"/>
+<junction x="-35.56" y="27.94"/>
 </segment>
 </net>
@@
 </segment>
 </net>
-<net name="AD3" class="0">
-<segment>
-<pinref part="X3" gate="-5" pin="1"/>
-<wire x1="-30.48" y1="7.62" x2="-35.56" y2="7.62" width="0.1524" layer="91"/>
-<label x="-35.306" y="8.382" size="1.778" layer="95"/>
-</segment>
-</net>
-<net name="AD4" class="0">
-<segment>
-<pinref part="X3" gate="-6" pin="1"/>
-<wire x1="-30.48" y1="2.54" x2="-35.56" y2="2.54" width="0.1524" layer="91"/>
-<label x="-35.306" y="3.302" size="1.778" layer="95"/>
-</segment>
-</net>
-<net name="AD5" class="0">
-<segment>
-<pinref part="X3" gate="-7" pin="1"/>
-<wire x1="-30.48" y1="-2.54" x2="-35.56" y2="-2.54" width="0.1524" layer="91"/>
-<label x="-35.56" y="-2.032" size="1.778" layer="95"/>
-</segment>
-</net>
-<net name="AD6" class="0">
-<segment>
-<pinref part="X3" gate="-8" pin="1"/>
-<wire x1="-30.48" y1="-7.62" x2="-35.56" y2="-7.62" width="0.1524" layer="91"/>
-<label x="-35.56" y="-6.858" size="1.778" layer="95"/>
-</segment>
-</net>
 <net name="AD7" class="0">
-<segment>
-<pinref part="X3" gate="-9" pin="1"/>
-<wire x1="-30.48" y1="-12.7" x2="-35.56" y2="-12.7" width="0.1524" layer="91"/>
-<label x="-35.56" y="-12.192" size="1.778" layer="95"/>
-</segment>
 <segment>
 <pinref part="X2" gate="-4" pin="1"/>
@@
 <label x="-78.486" y="12.954" size="1.778" layer="95"/>
 </segment>
+<segment>
+<pinref part="IC3" gate="PORTA_L" pin="PA5"/>
+<wire x1="-81.28" y1="-43.18" x2="-88.9" y2="-43.18" width="0.1524" layer="91"/>
+<label x="-90.932" y="-42.926" size="1.778" layer="95"/>
+</segment>
 </net>
 <net name="W_CLK" class="0">
@@
 <label x="-79.756" y="23.876" size="1.778" layer="95"/>
 </segment>
+<segment>
+<pinref part="IC3" gate="PORTA_L" pin="PA3"/>
+<wire x1="-81.28" y1="-38.1" x2="-88.9" y2="-38.1" width="0.1524" layer="91"/>
+<label x="-90.678" y="-37.592" size="1.778" layer="95"/>
+</segment>
 </net>
 <net name="FQ_UD" class="0">
@@
 <label x="-79.756" y="18.796" size="1.778" layer="95"/>
 </segment>
+<segment>
+<pinref part="IC3" gate="PORTA_L" pin="PA4"/>
+<wire x1="-81.28" y1="-40.64" x2="-88.9" y2="-40.64" width="0.1524" layer="91"/>
+<label x="-90.932" y="-40.132" size="1.778" layer="95"/>
+</segment>
 </net>
 <net name="A_RESET" class="0">
@@
 <wire x1="-71.12" y1="7.62" x2="-78.74" y2="7.62" width="0.1524" layer="91"/>
 <label x="-82.042" y="8.128" size="1.778" layer="95"/>
+</segment>
+<segment>
+<pinref part="IC3" gate="PORTA_L" pin="PA6"/>
+<wire x1="-81.28" y1="-45.72" x2="-88.9" y2="-45.72" width="0.1524" layer="91"/>
+<label x="-92.964" y="-45.466" size="1.778" layer="95"/>
 </segment>
 </net>
@@
 <wire x1="-66.04" y1="60.96" x2="-71.12" y2="60.96" width="0.1524" layer="91"/>
 <junction x="-71.12" y="60.96"/>
-<pinref part="X1" gate="G$1" pin="1"/>
 <wire x1="-71.12" y1="60.96" x2="-81.28" y2="60.96" width="0.1524" layer="91"/>
 <wire x1="-81.28" y1="60.96" x2="-81.28" y2="55.88" width="0.1524" layer="91"/>
+<pinref part="X1" gate="G$1" pin="1"/>
 </segment>
 </net>
@@
 </segment>
 </net>
+<net name="N$36" class="0">
+<segment>
+<pinref part="X3" gate="-9" pin="1"/>
+<wire x1="-30.48" y1="-12.7" x2="-35.56" y2="-12.7" width="0.1524" layer="91"/>
+</segment>
+</net>

Commit message: - ?????? ????????? ?????
Parts:
- removed C31, C32: 100n, rcl:C-EUC0603
- removed C35: 1mk, rcl:C-EUC0603
- C17, C18, C19, C20: device rcl:C-EUC0603 -> rcl:C-EUC0805
Connections:
- net +3V3: no longer C35.1
- net AD7: now also IC3PORTB_L.PB5; no longer IC3PORTA_L.PA5
- net A_RESET: now also IC3PORTB_L.PB6; no longer IC3PORTA_L.PA6
- net FQ_UD: now also IC3PORTB_L.PB4; no longer IC3PORTA_L.PA4
- net GND: no longer C31.2, C32.2, C35.2
- net N$15: no longer C31.1
- net N$23: no longer C32.1
- net W_CLK: now also IC3PORTB_L.PB3; no longer IC3PORTA_L.PA3

Commit message: - ????????? ??????????? AD9850 ??????
Parts:
- removed X5: SWD, con-cypressindustries:MINI-USB-SCHIELD-32005-301
- added C31: 100n, rcl:C-EUC0603
- added X6: (no value), con-phoenix-254:MPT4
Connections:
- net +3V3: now also X6-1.1; no longer X5G$1.1
- net +5V: now also C31.1
- net AD7: now also IC3PORTB_L.PB4; no longer IC3PORTB_L.PB5
- net A_RESET: now also IC3PORTB_L.PB3; no longer IC3PORTB_L.PB6
- net FQ_UD: now also IC3PORTB_L.PB5; no longer IC3PORTB_L.PB4
- net GND: now also C31.2, X6-4.1; no longer X5G$1.5, X5S.S1, X5S.S2, X5S.S3, X5S.S4
- net SWDCLK: now also X6-3.1; no longer X5G$1.3
- net SWDIO: now also X6-2.1; no longer X5G$1.2
- net W_CLK: now also IC3PORTB_L.PB6; no longer IC3PORTB_L.PB3

Commit message: - ??????? ?????? ?????????
Parts:
- removed C10: 100n, rcl:C-EUC0603
- added C32: 1mk, rcl:C-EUC0603
- added X5: (no value), con-phoenix-254:MPT4
Connections:
- new net N$38: C37.2, X5-1.1
- new net N$39: C38.2, X5-3.1
- net +5V: now also C32.1; no longer C10.1
- net GND: now also C32.2, X5-2.1, X5-4.1; no longer C10.2
Changed lines of the file:
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@@
 <part name="IC2" library="74xx-eu" deviceset="74*74" device="D" technology="AC"/>
 <part name="P+1" library="supply1" deviceset="+5V" device=""/>
-<part name="GND1" library="supply1" deviceset="GND" device=""/>
-<part name="C10" library="rcl" deviceset="C-EU" device="C0603" value="100n"/>
 <part name="R10" library="rcl" deviceset="R-EU_" device="R0603" value="10"/>
 <part name="R11" library="rcl" deviceset="R-EU_" device="R0603" value="10"/>
@@
 <part name="+3V5" library="supply1" deviceset="+3V3" device=""/>
 <part name="C31" library="rcl" deviceset="C-EU" device="C0603" value="100n"/>
+<part name="X5" library="con-phoenix-254" deviceset="MPT4" device=""/>
+<part name="GND13" library="supply1" deviceset="GND" device=""/>
+<part name="GND25" library="supply1" deviceset="GND" device=""/>
+<part name="C32" library="rcl" deviceset="C-EU" device="C0603" value="1mk"/>
+<part name="GND26" library="supply1" deviceset="GND" device=""/>
 </parts>
 <sheets>
@@
 <instance part="IC2" gate="P" x="93.98" y="-7.62"/>
 <instance part="P+1" gate="1" x="17.78" y="27.94"/>
-<instance part="GND1" gate="1" x="17.78" y="-22.86"/>
-<instance part="C10" gate="G$1" x="17.78" y="-15.24"/>
 <instance part="R10" gate="G$1" x="55.88" y="22.86"/>
 <instance part="R11" gate="G$1" x="55.88" y="-10.16"/>
@@
 <instance part="+3V5" gate="G$1" x="119.38" y="-48.26"/>
 <instance part="C31" gate="G$1" x="109.22" y="-7.62"/>
+<instance part="X5" gate="-1" x="167.64" y="76.2"/>
+<instance part="X5" gate="-2" x="167.64" y="71.12"/>
+<instance part="X5" gate="-3" x="167.64" y="66.04"/>
+<instance part="X5" gate="-4" x="167.64" y="60.96"/>
+<instance part="GND13" gate="1" x="162.56" y="55.88"/>
+<instance part="GND25" gate="1" x="160.02" y="68.58"/>
+<instance part="C32" gate="G$1" x="142.24" y="101.6" rot="R90"/>
+<instance part="GND26" gate="1" x="149.86" y="99.06"/>
 </instances>
 <busses>
@@
 <junction x="17.78" y="12.7"/>
 <junction x="17.78" y="22.86"/>
-<pinref part="C10" gate="G$1" pin="1"/>
-<wire x1="17.78" y1="-12.7" x2="17.78" y2="-10.16" width="0.1524" layer="91"/>
-<junction x="17.78" y="-10.16"/>
 </segment>
 <segment>
@@
 <wire x1="129.54" y1="99.06" x2="129.54" y2="101.6" width="0.1524" layer="91"/>
 <pinref part="P+2" gate="1" pin="+5V"/>
+<pinref part="C32" gate="G$1" pin="1"/>
+<wire x1="139.7" y1="101.6" x2="129.54" y2="101.6" width="0.1524" layer="91"/>
+<junction x="129.54" y="101.6"/>
 </segment>
 <segment>
@@
 </net>
 <net name="GND" class="0">
-<segment>
-<pinref part="C10" gate="G$1" pin="2"/>
-<pinref part="GND1" gate="1" pin="GND"/>
-</segment>
 <segment>
 <pinref part="IC5" gate="A" pin="V-"/>
@@
 <wire x1="119.38" y1="-68.58" x2="119.38" y2="-71.12" width="0.1524" layer="91"/>
 </segment>
+<segment>
+<pinref part="X5" gate="-2" pin="1"/>
+<pinref part="GND25" gate="1" pin="GND"/>
+<wire x1="165.1" y1="71.12" x2="160.02" y2="71.12" width="0.1524" layer="91"/>
+</segment>
+<segment>
+<pinref part="X5" gate="-4" pin="1"/>
+<pinref part="GND13" gate="1" pin="GND"/>
+<wire x1="165.1" y1="60.96" x2="162.56" y2="60.96" width="0.1524" layer="91"/>
+<wire x1="162.56" y1="60.96" x2="162.56" y2="58.42" width="0.1524" layer="91"/>
+</segment>
+<segment>
+<pinref part="GND26" gate="1" pin="GND"/>
+<pinref part="C32" gate="G$1" pin="2"/>
+<wire x1="149.86" y1="101.6" x2="147.32" y2="101.6" width="0.1524" layer="91"/>
+</segment>
 </net>
 <net name="N$1" class="0">
@@
 </segment>
 </net>
+<net name="N$38" class="0">
+<segment>
+<pinref part="C37" gate="G$1" pin="2"/>
+<wire x1="154.94" y1="91.44" x2="157.48" y2="91.44" width="0.1524" layer="91"/>
+<wire x1="157.48" y1="91.44" x2="157.48" y2="76.2" width="0.1524" layer="91"/>
+<pinref part="X5" gate="-1" pin="1"/>
+<wire x1="157.48" y1="76.2" x2="165.1" y2="76.2" width="0.1524" layer="91"/>
+</segment>
+</net>
+<net name="N$39" class="0">
+<segment>
+<pinref part="X5" gate="-3" pin="1"/>
+<wire x1="165.1" y1="66.04" x2="157.48" y2="66.04" width="0.1524" layer="91"/>
+<wire x1="157.48" y1="66.04" x2="157.48" y2="43.18" width="0.1524" layer="91"/>
+<pinref part="C38" gate="G$1" pin="2"/>
+<wire x1="157.48" y1="43.18" x2="154.94" y2="43.18" width="0.1524" layer="91"/>
+</segment>
+</net>

Commit message: - ?????? ???? ?????? ??????? ????? ??
Parts:
- removed C29, C30: 1mk, rcl:C-EUC0603
- removed R24, R25: 10K, rcl:R-EU_R0603
- R18, R19, R22, R23: value 10K -> 22K
Connections:
- removed net N$24: IC6.+IN, R21.2, R25.2
- removed net N$26: IC5.+IN, R17.2, R24.2
- net GND: no longer C29.2, C30.2
- net N$15: now also IC5.+IN, R17.2; no longer C29.1, R24.1
- net N$23: now also IC6.+IN, R21.2; no longer C30.1, R25.1

Commit message: - ??? ??????????????????. - ???????? ??????, ????? ???????? ????????????? ??????? ????????.
Parts:
- added X7: (no value), con-phoenix-254:MPT2
Connections:
- net AD7: now also IC3PORTA_L.PA4; no longer IC3PORTB_L.PB4
- net A_RESET: now also IC3PORTA_L.PA3; no longer IC3PORTB_L.PB3
- net FQ_UD: now also IC3PORTA_L.PA5; no longer IC3PORTB_L.PB5
- net I-LO: now also X7-1.1
- net Q-LO: now also X7-2.1
- net W_CLK: now also IC3PORTA_L.PA6; no longer IC3PORTB_L.PB6
Changed lines of the file:
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@@
 <part name="C32" library="rcl" deviceset="C-EU" device="C0603" value="1mk"/>
 <part name="GND26" library="supply1" deviceset="GND" device=""/>
+<part name="X7" library="con-phoenix-254" deviceset="MPT2" device=""/>
 </parts>
 <sheets>
@@
 <instance part="C32" gate="G$1" x="142.24" y="101.6" rot="R90"/>
 <instance part="GND26" gate="1" x="149.86" y="99.06"/>
+<instance part="X7" gate="-1" x="63.5" y="10.16"/>
+<instance part="X7" gate="-2" x="63.5" y="5.08"/>
 </instances>
 <busses>
@@
 <pinref part="IC1" gate="A" pin="C"/>
 <wire x1="68.58" y1="48.26" x2="48.26" y2="48.26" width="0.1524" layer="91"/>
+<pinref part="X7" gate="-1" pin="1"/>
+<wire x1="60.96" y1="10.16" x2="60.96" y2="22.86" width="0.1524" layer="91"/>
+<junction x="60.96" y="22.86"/>
 </segment>
 </net>
@@
 <pinref part="IC1" gate="A" pin="B"/>
 <wire x1="73.66" y1="50.8" x2="48.26" y2="50.8" width="0.1524" layer="91"/>
+<pinref part="X7" gate="-2" pin="1"/>
+<wire x1="60.96" y1="5.08" x2="60.96" y2="-10.16" width="0.1524" layer="91"/>
+<junction x="60.96" y="-10.16"/>
 </segment>
 </net>
@@
 </segment>
 <segment>
-<pinref part="IC3" gate="PORTB_L" pin="PB4"/>
-<wire x1="-48.26" y1="-40.64" x2="-43.18" y2="-40.64" width="0.1524" layer="91"/>
-<label x="-48.26" y="-40.64" size="1.778" layer="95"/>
+<pinref part="IC3" gate="PORTA_L" pin="PA4"/>
+<wire x1="-81.28" y1="-40.64" x2="-88.9" y2="-40.64" width="0.1524" layer="91"/>
 </segment>
 </net>
@@
 </segment>
 <segment>
-<pinref part="IC3" gate="PORTB_L" pin="PB6"/>
-<wire x1="-48.26" y1="-45.72" x2="-43.18" y2="-45.72" width="0.1524" layer="91"/>
-<label x="-48.26" y="-45.72" size="1.778" layer="95"/>
+<pinref part="IC3" gate="PORTA_L" pin="PA6"/>
+<wire x1="-81.28" y1="-45.72" x2="-88.9" y2="-45.72" width="0.1524" layer="91"/>
 </segment>
 </net>
@@
 </segment>
 <segment>
-<pinref part="IC3" gate="PORTB_L" pin="PB5"/>
-<wire x1="-48.26" y1="-43.18" x2="-43.18" y2="-43.18" width="0.1524" layer="91"/>
-<label x="-48.26" y="-43.18" size="1.778" layer="95"/>
+<pinref part="IC3" gate="PORTA_L" pin="PA5"/>
+<wire x1="-81.28" y1="-43.18" x2="-88.9" y2="-43.18" width="0.1524" layer="91"/>
 </segment>
 </net>
@@
 </segment>
 <segment>
-<pinref part="IC3" gate="PORTB_L" pin="PB3"/>
-<wire x1="-48.26" y1="-38.1" x2="-43.18" y2="-38.1" width="0.1524" layer="91"/>
-<label x="-48.26" y="-38.1" size="1.778" layer="95"/>
-</segment>
-</net>
+<pinref part="IC3" gate="PORTA_L" pin="PA3"/>
+<wire x1="-81.28" y1="-38.1" x2="-88.9" y2="-38.1" width="0.1524" layer="91"/>
+</segment>
+</net>
