File: circuit/mini.sch (EAGLE design)
At the start: 79 parts, among them IC1 74AC4053D, IC2 74AC74D, IC3 STM32L151CBT6, IC4 MCP1700-3.3V, IC5 NE5534D, IC6 NE5534D, Q1 BFG135, Q2 8MHz, X1 1-227161-0, X4 MINI-USB

Commit message: - ????????? ????? - ?????????? ?????????? ?????? ??? IC5
Connections:
- net N$10: now also IC1A.Y1; no longer IC1A.Y0
- net N$9: now also IC1A.Y0; no longer IC1A.Y1
Changed lines of the file:
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@@
-</segment>
-</net>
-<net name="N$9" class="0">
-<segment>
-<pinref part="IC1" gate="A" pin="Y1"/>
-<wire x1="48.26" y1="68.58" x2="58.42" y2="68.58" width="0.1524" layer="91"/>
-<wire x1="58.42" y1="68.58" x2="58.42" y2="86.36" width="0.1524" layer="91"/>
-<pinref part="R13" gate="G$1" pin="1"/>
-<wire x1="58.42" y1="86.36" x2="60.96" y2="86.36" width="0.1524" layer="91"/>
-</segment>
-</net>
-<net name="N$10" class="0">
-<segment>
-<pinref part="IC1" gate="A" pin="Y0"/>
-<wire x1="48.26" y1="71.12" x2="55.88" y2="71.12" width="0.1524" layer="91"/>
-<wire x1="55.88" y1="71.12" x2="55.88" y2="93.98" width="0.1524" layer="91"/>
-<pinref part="R12" gate="G$1" pin="1"/>
-<wire x1="55.88" y1="93.98" x2="60.96" y2="93.98" width="0.1524" layer="91"/>
 </segment>
 </net>
@@
 </segment>
 </net>
+<net name="N$9" class="0">
+<segment>
+<pinref part="IC1" gate="A" pin="Y0"/>
+<pinref part="R13" gate="G$1" pin="1"/>
+<wire x1="48.26" y1="71.12" x2="60.96" y2="71.12" width="0.1524" layer="91"/>
+<wire x1="60.96" y1="71.12" x2="60.96" y2="86.36" width="0.1524" layer="91"/>
+</segment>
+</net>
+<net name="N$10" class="0">
+<segment>
+<pinref part="R12" gate="G$1" pin="1"/>
+<wire x1="60.96" y1="93.98" x2="55.88" y2="93.98" width="0.1524" layer="91"/>
+<wire x1="55.88" y1="93.98" x2="55.88" y2="68.58" width="0.1524" layer="91"/>
+<pinref part="IC1" gate="A" pin="Y1"/>
+<wire x1="55.88" y1="68.58" x2="48.26" y2="68.58" width="0.1524" layer="91"/>
+</segment>
+</net>
