File: circuit/dds_ad9958.brd (EAGLE design)
At the start: 100 x 80 mm, 68 parts, among them IC1 TPS76833, IC2 TPS79318, IC3 TPS79318, IC4 AD9958, Q1 25MHz, X2 BU-SMA-V, X3 BU-SMA-V

Commit message: - ??????? ?????????
Parts:
- moved C29 28.0 mm to (25.4, 13.4), turned to 180 degrees
- moved C30 26.5 mm to (19.6, 13.4), turned to 180 degrees
- moved L6 26.5 mm to (25.4, 10.1), turned to 180 degrees
- moved L7 26.0 mm to (19.6, 10.1), turned to 180 degrees
- moved L8 25.0 mm to (13.5, 10.1), turned to 180 degrees
- moved C31 25.0 mm to (13.5, 13.4), turned to 180 degrees
- moved X3 23.0 mm to (6.08, 12.8)
- moved C37 23.0 mm to (11.9, 17.4), turned to 90 degrees
- moved C10 21.6 mm to (72.4, 25.4)
- moved C11 21.6 mm to (72.4, 28.0)
- moved C17 21.6 mm to (51.7, 24.8)
- moved C20 21.6 mm to (65.0, 26.8)
- moved IC4 21.6 mm to (59.5, 22.9)
- moved L2 21.6 mm to (70.5, 16.1)
- moved L3 21.6 mm to (25.7, 25.4)
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Routing:
- net AVDD: track 104.3 -> 168.3 mm, vias 2 -> 5
- net GND: track 271.0 -> 328.7 mm
- net N$24: track 0.00 -> 14.1 mm
- net N$25: track 0.00 -> 13.3 mm
- net N$26: track 0.00 -> 12.8 mm
- net N$23: track 0.00 -> 12.3 mm
Other:
- board size 100 x 80 mm -> 84 x 40.5 mm

Commit message: - ??????? ? ????????? ????????
Parts:
- L3, L4, L5, L6, L7, L8: device rcl:L3225P -> rcl:C0805
- moved L4 8.14 mm to (21.3, 33.4), flipped to the bottom, turned to 45 degrees
- moved L3 7.50 mm to (25.7, 32.9), flipped to the bottom, turned to 315 degrees
- moved L5 6.67 mm to (15.5, 31.9), flipped to the bottom, turned to 315 degrees
- moved C27 5.85 mm to (13.1, 26.7), flipped to the bottom, turned to 270 degrees
- moved C26 5.70 mm to (17.5, 26.8), flipped to the bottom, turned to 270 degrees
- moved C24 5.59 mm to (27.4, 26.8), flipped to the bottom, turned to 270 degrees
- moved C25 5.50 mm to (21.8, 26.8), flipped to the bottom, turned to 270 degrees
- moved C23 4.50 mm to (14.0, 33.2), flipped to the bottom, turned to 315 degrees
- moved R11 4.03 mm to (46.0, 18.4), flipped to the bottom, turned to 90 degrees
- moved R8 4.00 mm to (47.0, 26.0), flipped to the bottom, turned to 270 degrees
- moved L6 3.61 mm to (27.4, 13.1), flipped to the bottom, turned to 315 degrees
- moved R14 3.54 mm to (46.0, 14.3), flipped to the bottom, turned to 270 degrees
- moved X2 3.54 mm to (6.08, 31.6)
- moved C22 3.50 mm to (19.8, 32.2), flipped to the bottom, turned to 45 degrees
- moved C21 3.20 mm to (27.2, 31.2), flipped to the bottom, turned to 315 degrees
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Routing:
- net AVDD: track 168.3 -> 145.9 mm, vias 5 -> 6
- net GND: track 328.7 -> 342.5 mm, vias 3 -> 6
- net N$7: track 28.6 -> 15.6 mm, vias 0 -> 1
- net N$9: track 20.2 -> 13.0 mm, vias 2 -> 1
- net N$3: track 16.5 -> 21.4 mm, vias 0 -> 1
- net N$10: track 12.9 -> 16.8 mm, vias 0 -> 1
- net N$26: track 12.8 -> 15.2 mm, vias 0 -> 1
- net N$25: track 13.3 -> 15.5 mm
- net N$23: track 12.3 -> 10.4 mm
- net N$11: track 13.0 -> 11.8 mm
- net N$6: track 26.7 -> 27.8 mm
- net N$2: track 11.6 -> 10.5 mm
- net N$18: track 13.1 -> 12.3 mm
- net N$24: track 14.1 -> 13.6 mm
- net N$20: track 13.9 -> 14.0 mm, vias 0 -> 1
- added copper zone on layer 1, net GND
- added copper zone on layer 16, net GND

Commit message: - ????????? ????????? ????? ?????????? ?????
Parts:
- L1, L2: device rcl:L3225P -> rcl:C0805
- moved C23 0.25 mm to (14.0, 33.4)
- moved L4 0.25 mm to (21.3, 33.6)
Routing:
- net N$33: track 0.00 -> 4.00 mm
- net N$31: track 0.00 -> 4.00 mm
- net N$19: track 0.00 -> 4.00 mm
- net N$37: track 0.00 -> 3.50 mm
- net N$36: track 0.00 -> 3.50 mm
- net N$34: track 0.00 -> 3.50 mm
- net N$14: track 0.00 -> 3.50 mm
- net N$35: track 0.00 -> 3.00 mm
- net GND: track 342.5 -> 340.3 mm, vias 6 -> 10
Other:
- board size 84 x 40.5 mm -> 84 x 40 mm

Commit message: - CS4272 test board
Connections:
- net N$13 renamed SDIO_1
- net N$21 renamed SDIO_2
- net N$22 renamed SDIO_3
Changed lines of the file:
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@@
 <layer number="18" name="Vias" color="2" fill="1" visible="yes" active="yes"/>
 <layer number="19" name="Unrouted" color="6" fill="1" visible="yes" active="yes"/>
-<layer number="20" name="Dimension" color="15" fill="1" visible="no" active="yes"/>
-<layer number="21" name="tPlace" color="7" fill="1" visible="no" active="yes"/>
+<layer number="20" name="Dimension" color="15" fill="1" visible="yes" active="yes"/>
+<layer number="21" name="tPlace" color="7" fill="1" visible="yes" active="yes"/>
 <layer number="22" name="bPlace" color="7" fill="1" visible="no" active="yes"/>
 <layer number="23" name="tOrigins" color="15" fill="1" visible="no" active="yes"/>
@@
 <wire x1="69.57" y1="33.07" x2="69.5" y2="33" width="0.25" layer="1"/>
 </signal>
-<signal name="N$13">
+<signal name="SDIO_1">
 <contactref element="IC4" pad="P$51"/>
 <contactref element="R9" pad="2"/>
@@
 <wire x1="58.71" y1="32.04" x2="60.41" y2="33.74" width="0.25" layer="1"/>
 </signal>
-<signal name="N$21">
+<signal name="SDIO_2">
 <contactref element="IC4" pad="P$52"/>
 <contactref element="R12" pad="2"/>
@@
 <wire x1="58.21" y1="33.62" x2="58.35" y2="33.76" width="0.25" layer="1"/>
 </signal>
-<signal name="N$22">
+<signal name="SDIO_3">
 <contactref element="IC4" pad="P$53"/>
 <contactref element="R13" pad="2"/>
