File: circuit/dds_ad9958.sch (EAGLE design)
At the start: 67 parts, among them IC1 AD9958, IC2 TPS79318, IC3 TPS76833, IC4 TPS79318, Q1 25MHz, X1 BU-SMA-V, X2 BU-SMA-V

Commit message: - renumber
Parts:
- added C36: 27pF, rcl:C-EUC0805
- added C37: 12pF, rcl:C-EUC0805
- C1, C2: value 22 -> 10u; device rcl:C-EUC0603 -> rcl:C-EUC0805
- C10, C11, C12, C13, C9: value 100n -> 47pF; device rcl:C-EUC0603 -> rcl:C-EUC0805
- C15: value 22pF -> 100n; device rcl:C-EUC0805 -> rcl:C-EUC0603
- C16: value 33pF -> 100n; device rcl:C-EUC0805 -> rcl:C-EUC0603
- C17: value 27pF -> 100n; device rcl:C-EUC0805 -> rcl:C-EUC0603
- C18, C28: value 12pF -> 100n; device rcl:C-EUC0805 -> rcl:C-EUC0603
- C19: value 2.2pF -> 100n; device rcl:C-EUC0805 -> rcl:C-EUC0603
- C20: value 6.8pF -> 100n; device rcl:C-EUC0805 -> rcl:C-EUC0603
- C21: value 12pF -> 2.2pF
- C22: value 22pF -> 6.8pF
- C23: value 33pF -> 12pF
- C24: value 27pF -> 22pF
- C25: value 12pF -> 33pF
- C26: value 2.2pF -> 27pF
- C27: value 6.8pF -> 12pF
- C29: value 1u -> 2.2pF; device rcl:C-EUC0603 -> rcl:C-EUC0805
- C3: value 1u -> 10u; device rcl:C-EUC0603 -> rcl:C-EUC0805
- C30: value 47pF -> 6.8pF
- C31: value 47pF -> 12pF
- C32, C33: value 47pF -> 22; device rcl:C-EUC0805 -> rcl:C-EUC0603
- C34: value 47pF -> 22pF
- C35: value 100n -> 33pF; device rcl:C-EUC0603 -> rcl:C-EUC0805
- C5: value 100n -> 1u
- C7: value 10u -> 1u; device rcl:C-EUC0805 -> rcl:C-EUC0603
- C8: value 10u -> 100n; device rcl:C-EUC0805 -> rcl:C-EUC0603
- IC1: value AD9958 -> TPS76833; device balmer:AD9958 -> balmer:TPS768XX
- IC3: value TPS76833 -> TPS79318; device balmer:TPS768XX -> balmer:TPS793XX_FIXED
- IC4: value TPS79318 -> AD9958; device balmer:TPS793XX_FIXED -> balmer:AD9958
- R1: value 2.2K -> 47
- R10: value 47 -> 2.2K
- R11, R14: value 47 -> 120
- R12, R13: value 47 -> 10K
- R2, R3, R4, R5: value 10K -> 47
- R6, R9: value 120 -> 10K
- X1: value BU-SMA-V -> (none); device con-coax:BU-SMA-V -> con-phoenix-254:MPT8
- X3: value (none) -> BU-SMA-V; device con-phoenix-254:MPT8 -> con-coax:BU-SMA-V
Connections:
- net +3V3: now also C1.1, C28.1, C5.1, C7.1, IC1.OUT, IC3.EN, IC3.IN, IC4.DVDD_I_O; no longer C3.1, C35.1, C4.1, IC1.DVDD_I_O, IC3.OUT, IC4.EN, IC4.IN
- net CS: now also C11.1, IC4.CS, R3.1; no longer C31.1, IC1.CS, R12.1
- net GND: now also C19.2, C20.2, C26.2, C27.2, C28.2, C36.2, C37.2, IC1.EN_, IC1.GND, IC4.AGND, IC4.DGND, IC4.P0, IC4.P1, IC4.P2, IC4.P3, IC4.PWR_DWN_CTL, R10.2, R12.1, R13.1, R6.2, R9.1, X1-2.1, X1-3.1, X3.2; no longer C22.2, C23.2, C29.2, C30.2, C31.2, IC1.AGND, IC1.DGND, IC1.P0, IC1.P1, IC1.P2, IC1.P3, IC1.PWR_DWN_CTL, IC3.EN_, IC4.GND, R1.2, R2.2, R3.1, R4.1, R5.1, X1.2, X3-2.1, X3-3.1
- net I_O_UPDATE: now also C10.1, IC4.I_O_UPDATE, R2.1; no longer C32.1, IC1.I_O_UPDATE, R11.1
- net MASTER_RESET: now also C9.1, IC4.MASTER_RESET, R1.1; no longer C33.1, IC1.MASTER_RESET, R10.1
- net N$1: now also C32.1, IC4.REF_CLK_N; no longer C1.1, IC1.REF_CLK_N
- net N$10: now also IC4.CH1_IOUT_N, R14.2; no longer IC1.CH1_IOUT_N, R9.2
- net N$11: now also C21.2, C22.1, C25.1; no longer C16.1, C19.2, C20.1
- net N$12: now also IC4.DAC_RSET, R10.1; no longer IC1.DAC_RSET, R1.1
- net N$13: now also IC4.SDIO_1, R9.2; no longer IC1.SDIO_1, R3.2
- net N$14: now also C19.1, C20.1, IC4.DVDD, L1.2; no longer C13.1, IC1.DVDD, L2.2
- net N$15: now also IC4.SYNC_IN, R6.1; no longer IC1.SYNC_IN, R2.1
- net N$16: now also IC4.LOOP_FILTER; no longer IC1.LOOP_FILTER
- net N$17: now also C33.1, IC4.REF_CLK; no longer C2.1, IC1.REF_CLK
- net N$18: now also C22.2, C23.1, C26.1; no longer C17.1, C20.2, C21.1
- net N$19: now also C15.1, C16.1, C17.1, C18.1, IC4.AVDD, IC4.CLK_MODE_SEL, L2.2, R11.1, R14.1; no longer C10.1, C11.1, C12.1, C9.1, IC1.AVDD, IC1.CLK_MODE_SEL, L1.2, R6.1, R9.1
- net N$2: now also C21.1, C24.1; no longer C15.1, C19.1
- net N$20: now also C23.2, C27.1, X2.1; no longer C18.1, C21.2, X1.1
- net N$21: now also IC4.SDIO_2, R12.2; no longer IC1.SDIO_2, R4.2
- net N$22: now also IC4.SDIO_3, R13.2; no longer IC1.SDIO_3, R5.2
- net N$23: now also C29.1, C34.1; no longer C22.1, C26.1
- net N$24: now also C29.2, C30.1, C35.1; no longer C23.1, C26.2, C27.1
- net N$25: now also C30.2, C31.1, C36.1; no longer C24.1, C27.2, C28.1
- net N$26: now also C31.2, C37.1, X3.1; no longer C25.1, C28.2, X2.1
- net N$27: now also R3.2, X1-6.1; no longer R12.2, X3-6.1
- net N$28: now also R5.2, X1-8.1; no longer R14.2, X3-8.1
- net N$29: now also R1.2, X1-4.1; no longer R10.2, X3-4.1
- net N$3: now also IC4.CH0_IOUT, R7.2; no longer IC1.CH0_IOUT, R6.2
- net N$30: now also R2.2, X1-5.1; no longer R11.2, X3-5.1
- net N$32: now also R4.2, X1-7.1; no longer R13.2, X3-7.1
- net N$4: now also C6.1; no longer C5.1
- net N$5: now also C8.1, IC3.NR; no longer C6.1, IC4.NR
- net N$6: now also C2.1, L2.1; no longer C7.1, L1.1
- net N$7: now also IC4.CH0_IOUT_N, R8.2; no longer IC1.CH0_IOUT_N, R7.2
- net N$8: now also C3.1, IC3.OUT, L1.1; no longer C8.1, IC4.OUT, L2.1
- net N$9: now also IC4.CH1_IOUT, R11.2; no longer IC1.CH1_IOUT, R8.2
- net SCK: now also C12.1, IC4.SCLK, R4.1; no longer C30.1, IC1.SCLK, R13.1
- net SDIO_0: now also C13.1, IC4.SDIO_0, R5.1; no longer C34.1, IC1.SDIO_0, R14.1
- net VCC: now also C4.1, IC1.IN, X1-1.1; no longer C29.1, IC3.IN, X3-1.1
Other:
- moved on the sheet: C1, C10, C11, C12, C13, C15, C16, C17, C18, C19, C2, C20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

Commit message: - ???????? ??????? AD9958
Parts:
- removed C5: 1u, rcl:C-EUC0603
Connections:
- net N$14 renamed DVDD
- removed net N$19: C14.2, C15.1, C16.1, C17.1, C18.1, IC4.AVDD, IC4.CLK_MODE_SEL, L2.2, R11.1, R14.1, R7.1, R8.1, TR1.SEC, TR2.SEC
- new net AVDD: C14.2, C15.1, C16.1, C17.1, C18.1, IC4.AVDD, IC4.CLK_MODE_SEL, L2.2, R11.1, R14.1, R7.1, R8.1, TR1.SEC_CT, TR2.SEC_CT
- net +3V3: no longer C5.1
- net GND: no longer C5.2
- net N$10: now also TR2.SEC; no longer TR2.SEC_CT
- net N$7: now also TR1.SEC; no longer TR1.SEC_CT
Changed lines of the file:
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@@
 <part name="GND2" library="supply1" deviceset="GND" device=""/>
 <part name="+3V1" library="supply1" deviceset="+3V3" device=""/>
-<part name="C5" library="rcl" deviceset="C-EU" device="C0603" value="1u"/>
 <part name="GND3" library="supply1" deviceset="GND" device=""/>
 <part name="C7" library="rcl" deviceset="C-EU" device="C0603" value="1u"/>
@@
 <instance part="GND2" gate="1" x="22.86" y="88.9"/>
 <instance part="+3V1" gate="G$1" x="38.1" y="111.76"/>
-<instance part="C5" gate="G$1" x="48.26" y="96.52"/>
 <instance part="GND3" gate="1" x="66.04" y="88.9"/>
 <instance part="C7" gate="G$1" x="96.52" y="96.52"/>
@@
 </segment>
 <segment>
-<pinref part="C5" gate="G$1" pin="2"/>
 <pinref part="IC2" gate="G$1" pin="GND"/>
-<wire x1="48.26" y1="91.44" x2="66.04" y2="91.44" width="0.1524" layer="91"/>
 <pinref part="GND3" gate="1" pin="GND"/>
 <junction x="66.04" y="91.44"/>
@@
 <junction x="53.34" y="106.68"/>
 <junction x="101.6" y="106.68"/>
-<pinref part="C5" gate="G$1" pin="1"/>
-<wire x1="53.34" y1="99.06" x2="48.26" y2="99.06" width="0.1524" layer="91"/>
 <pinref part="C7" gate="G$1" pin="1"/>
 <wire x1="96.52" y1="99.06" x2="101.6" y2="99.06" width="0.1524" layer="91"/>
 <junction x="101.6" y="99.06"/>
-<junction x="53.34" y="99.06"/>
 <pinref part="C1" gate="G$1" pin="1"/>
 <junction x="40.64" y="106.68"/>
@@
 <wire x1="99.06" y1="58.42" x2="99.06" y2="40.64" width="0.1524" layer="91"/>
 <pinref part="TR1" gate="G$1" pin="SEC_DOT"/>
-<wire x1="116.84" y1="53.34" x2="119.38" y2="53.34" width="0.1524" layer="91"/>
+<wire x1="119.38" y1="53.34" x2="116.84" y2="53.34" width="0.1524" layer="91"/>
 <junction x="116.84" y="53.34"/>
 </segment>
@@
 <pinref part="IC4" gate="G$1" pin="CH0_IOUT_N"/>
 <wire x1="60.96" y1="38.1" x2="116.84" y2="38.1" width="0.1524" layer="91"/>
-<pinref part="TR1" gate="G$1" pin="SEC_CT"/>
 <pinref part="R8" gate="G$1" pin="2"/>
+<wire x1="116.84" y1="38.1" x2="116.84" y2="43.18" width="0.1524" layer="91"/>
+<pinref part="TR1" gate="G$1" pin="SEC"/>
 <wire x1="119.38" y1="43.18" x2="116.84" y2="43.18" width="0.1524" layer="91"/>
-<wire x1="116.84" y1="38.1" x2="116.84" y2="43.18" width="0.1524" layer="91"/>
-<junction x="116.84" y="43.18"/>
 </segment>
 </net>
@@
 <pinref part="IC4" gate="G$1" pin="CH1_IOUT"/>
 <wire x1="60.96" y1="35.56" x2="116.84" y2="35.56" width="0.1524" layer="91"/>
+<pinref part="R11" gate="G$1" pin="2"/>
+<wire x1="116.84" y1="35.56" x2="116.84" y2="25.4" width="0.1524" layer="91"/>
 <pinref part="TR2" gate="G$1" pin="SEC_DOT"/>
-<pinref part="R11" gate="G$1" pin="2"/>
-<wire x1="119.38" y1="25.4" x2="116.84" y2="25.4" width="0.1524" layer="91"/>
-<wire x1="116.84" y1="35.56" x2="116.84" y2="25.4" width="0.1524" layer="91"/>
+<wire x1="116.84" y1="25.4" x2="119.38" y2="25.4" width="0.1524" layer="91"/>
 <junction x="116.84" y="25.4"/>
 </segment>
@@
 <wire x1="60.96" y1="33.02" x2="104.14" y2="33.02" width="0.1524" layer="91"/>
 <wire x1="104.14" y1="33.02" x2="104.14" y2="10.16" width="0.1524" layer="91"/>
-<pinref part="TR2" gate="G$1" pin="SEC_CT"/>
 <pinref part="R14" gate="G$1" pin="2"/>
-<wire x1="119.38" y1="15.24" x2="116.84" y2="15.24" width="0.1524" layer="91"/>
 <wire x1="104.14" y1="10.16" x2="116.84" y2="10.16" width="0.1524" layer="91"/>
 <wire x1="116.84" y1="10.16" x2="116.84" y2="15.24" width="0.1524" layer="91"/>
-<junction x="116.84" y="15.24"/>
-</segment>
-</net>
-<net name="N$14" class="0">
+<pinref part="TR2" gate="G$1" pin="SEC"/>
+<wire x1="116.84" y1="15.24" x2="119.38" y2="15.24" width="0.1524" layer="91"/>
+</segment>
+</net>
+<net name="DVDD" class="0">
 <segment>
 <pinref part="IC4" gate="G$1" pin="DVDD"/>
@@
 <pinref part="C19" gate="G$1" pin="1"/>
 <junction x="132.08" y="76.2"/>
+<label x="124.46" y="76.2" size="1.778" layer="95"/>
 </segment>
 </net>
@@
 </segment>
 </net>
-<net name="N$19" class="0">
-<segment>
-<pinref part="R11" gate="G$1" pin="1"/>
-<wire x1="106.68" y1="25.4" x2="106.68" y2="20.32" width="0.1524" layer="91"/>
-<pinref part="TR2" gate="G$1" pin="SEC"/>
-<wire x1="106.68" y1="20.32" x2="119.38" y2="20.32" width="0.1524" layer="91"/>
-<pinref part="R14" gate="G$1" pin="1"/>
-<wire x1="106.68" y1="20.32" x2="106.68" y2="15.24" width="0.1524" layer="91"/>
-<pinref part="R7" gate="G$1" pin="1"/>
-<wire x1="106.68" y1="53.34" x2="106.68" y2="48.26" width="0.1524" layer="91"/>
-<pinref part="TR1" gate="G$1" pin="SEC"/>
-<wire x1="106.68" y1="48.26" x2="119.38" y2="48.26" width="0.1524" layer="91"/>
-<pinref part="R8" gate="G$1" pin="1"/>
-<wire x1="106.68" y1="48.26" x2="106.68" y2="43.18" width="0.1524" layer="91"/>
-<junction x="106.68" y="48.26"/>
+<net name="AVDD" class="0">
+<segment>
 <pinref part="L2" gate="G$1" pin="2"/>
 <pinref part="C15" gate="G$1" pin="1"/>
@@
 <wire x1="20.32" y1="68.58" x2="20.32" y2="76.2" width="0.1524" layer="91"/>
 <junction x="20.32" y="76.2"/>
+<label x="76.2" y="76.2" size="1.778" layer="95"/>
+<pinref part="R14" gate="G$1" pin="1"/>
+<pinref part="R11" gate="G$1" pin="1"/>
+<wire x1="106.68" y1="25.4" x2="106.68" y2="20.32" width="0.1524" layer="91"/>
+<wire x1="106.68" y1="20.32" x2="106.68" y2="15.24" width="0.1524" layer="91"/>
+<pinref part="TR2" gate="G$1" pin="SEC_CT"/>
+<wire x1="119.38" y1="20.32" x2="106.68" y2="20.32" width="0.1524" layer="91"/>
+<pinref part="R8" gate="G$1" pin="1"/>
+<pinref part="R7" gate="G$1" pin="1"/>
+<wire x1="106.68" y1="53.34" x2="106.68" y2="48.26" width="0.1524" layer="91"/>
+<wire x1="106.68" y1="48.26" x2="106.68" y2="43.18" width="0.1524" layer="91"/>
+<pinref part="TR1" gate="G$1" pin="SEC_CT"/>
+<wire x1="119.38" y1="48.26" x2="106.68" y2="48.26" width="0.1524" layer="91"/>
+<wire x1="119.38" y1="20.32" x2="119.38" y2="48.26" width="0.1524" layer="91"/>
 <wire x1="119.38" y1="48.26" x2="119.38" y2="76.2" width="0.1524" layer="91"/>
+<junction x="106.68" y="48.26"/>
 <junction x="119.38" y="48.26"/>
-<wire x1="119.38" y1="20.32" x2="119.38" y2="48.26" width="0.1524" layer="91"/>
 <junction x="119.38" y="20.32"/>
 <junction x="106.68" y="20.32"/>

Commit message: - ??????? ? ????????? ????????
Parts:
- L3, L4, L5, L6, L7, L8: device rcl:L-USL3225P -> rcl:L-USL0805
Changed lines of the file:
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@@
 <grid distance="0.1" unitdist="inch" unit="inch" style="lines" multiple="1" display="no" altdistance="0.01" altunitdist="inch" altunit="inch"/>
 <layers>
-<layer number="1" name="Top" color="4" fill="1" visible="no" active="no"/>
-<layer number="16" name="Bottom" color="1" fill="1" visible="no" active="no"/>
-<layer number="17" name="Pads" color="2" fill="1" visible="no" active="no"/>
-<layer number="18" name="Vias" color="2" fill="1" visible="no" active="no"/>
-<layer number="19" name="Unrouted" color="6" fill="1" visible="no" active="no"/>
-<layer number="20" name="Dimension" color="15" fill="1" visible="no" active="no"/>
-<layer number="21" name="tPlace" color="7" fill="1" visible="no" active="no"/>
-<layer number="22" name="bPlace" color="7" fill="1" visible="no" active="no"/>
-<layer number="23" name="tOrigins" color="15" fill="1" visible="no" active="no"/>
-<layer number="24" name="bOrigins" color="15" fill="1" visible="no" active="no"/>
-<layer number="25" name="tNames" color="7" fill="1" visible="no" active="no"/>
-<layer number="26" name="bNames" color="7" fill="1" visible="no" active="no"/>
-<layer number="27" name="tValues" color="7" fill="1" visible="no" active="no"/>
-<layer number="28" name="bValues" color="7" fill="1" visible="no" active="no"/>
+<layer number="1" name="Top" color="4" fill="1" visible="yes" active="no"/>
+<layer number="16" name="Bottom" color="1" fill="1" visible="yes" active="no"/>
+<layer number="17" name="Pads" color="2" fill="1" visible="yes" active="no"/>
+<layer number="18" name="Vias" color="2" fill="1" visible="yes" active="no"/>
+<layer number="19" name="Unrouted" color="6" fill="1" visible="yes" active="no"/>
+<layer number="20" name="Dimension" color="15" fill="1" visible="yes" active="no"/>
+<layer number="21" name="tPlace" color="7" fill="1" visible="yes" active="no"/>
+<layer number="22" name="bPlace" color="7" fill="1" visible="yes" active="no"/>
+<layer number="23" name="tOrigins" color="15" fill="1" visible="yes" active="no"/>
+<layer number="24" name="bOrigins" color="15" fill="1" visible="yes" active="no"/>
+<layer number="25" name="tNames" color="7" fill="1" visible="yes" active="no"/>
+<layer number="26" name="bNames" color="7" fill="1" visible="yes" active="no"/>
+<layer number="27" name="tValues" color="7" fill="1" visible="yes" active="no"/>
+<layer number="28" name="bValues" color="7" fill="1" visible="yes" active="no"/>
 <layer number="29" name="tStop" color="7" fill="3" visible="no" active="no"/>
 <layer number="30" name="bStop" color="7" fill="6" visible="no" active="no"/>
@@
 <layer number="35" name="tGlue" color="7" fill="4" visible="no" active="no"/>
 <layer number="36" name="bGlue" color="7" fill="5" visible="no" active="no"/>
-<layer number="37" name="tTest" color="7" fill="1" visible="no" active="no"/>
-<layer number="38" name="bTest" color="7" fill="1" visible="no" active="no"/>
+<layer number="37" name="tTest" color="7" fill="1" visible="yes" active="no"/>
+<layer number="38" name="bTest" color="7" fill="1" visible="yes" active="no"/>
 <layer number="39" name="tKeepout" color="4" fill="11" visible="no" active="no"/>
 <layer number="40" name="bKeepout" color="1" fill="11" visible="no" active="no"/>
@@
 <layer number="44" name="Drills" color="7" fill="1" visible="no" active="no"/>
 <layer number="45" name="Holes" color="7" fill="1" visible="no" active="no"/>
-<layer number="46" name="Milling" color="3" fill="1" visible="no" active="no"/>
-<layer number="47" name="Measures" color="7" fill="1" visible="no" active="no"/>
-<layer number="48" name="Document" color="7" fill="1" visible="no" active="no"/>
-<layer number="49" name="Reference" color="7" fill="1" visible="no" active="no"/>
-<layer number="50" name="dxf" color="7" fill="1" visible="no" active="no"/>
-<layer number="51" name="tDocu" color="7" fill="1" visible="no" active="no"/>
-<layer number="52" name="bDocu" color="7" fill="1" visible="no" active="no"/>
-<layer number="53" name="tGND_GNDA" color="7" fill="9" visible="no" active="no"/>
-<layer number="54" name="bGND_GNDA" color="1" fill="9" visible="no" active="no"/>
-<layer number="56" name="wert" color="7" fill="1" visible="no" active="no"/>
+<layer number="46" name="Milling" color="3" fill="1" visible="yes" active="no"/>
+<layer number="47" name="Measures" color="7" fill="1" visible="yes" active="no"/>
+<layer number="48" name="Document" color="7" fill="1" visible="yes" active="no"/>
+<layer number="49" name="Reference" color="7" fill="1" visible="yes" active="no"/>
+<layer number="50" name="dxf" color="7" fill="1" visible="yes" active="no"/>
+<layer number="51" name="tDocu" color="7" fill="1" visible="yes" active="no"/>
+<layer number="52" name="bDocu" color="7" fill="1" visible="yes" active="no"/>
+<layer number="53" name="tGND_GNDA" color="7" fill="9" visible="yes" active="no"/>
+<layer number="54" name="bGND_GNDA" color="1" fill="9" visible="yes" active="no"/>
+<layer number="56" name="wert" color="7" fill="1" visible="yes" active="no"/>
 <layer number="91" name="Nets" color="2" fill="1" visible="yes" active="yes"/>
 <layer number="92" name="Busses" color="1" fill="1" visible="yes" active="yes"/>
@@
 <part name="R11" library="rcl" deviceset="R-EU_" device="R0603" value="120"/>
 <part name="R14" library="rcl" deviceset="R-EU_" device="R0603" value="120"/>
-<part name="L3" library="rcl" deviceset="L-US" device="L3225P" value="68nH"/>
-<part name="L4" library="rcl" deviceset="L-US" device="L3225P" value="56nH"/>
-<part name="L5" library="rcl" deviceset="L-US" device="L3225P" value="39nH"/>
+<part name="L3" library="rcl" deviceset="L-US" device="L0805" value="68nH"/>
+<part name="L4" library="rcl" deviceset="L-US" device="L0805" value="56nH"/>
+<part name="L5" library="rcl" deviceset="L-US" device="L0805" value="39nH"/>
 <part name="C24" library="rcl" deviceset="C-EU" device="C0805" value="22pF"/>
 <part name="C25" library="rcl" deviceset="C-EU" device="C0805" value="33pF"/>
@@
 <part name="GND13" library="supply1" deviceset="GND" device=""/>
 <part name="X2" library="con-coax" deviceset="BU-SMA-V" device=""/>
-<part name="L6" library="rcl" deviceset="L-US" device="L3225P" value="68nH"/>
-<part name="L7" library="rcl" deviceset="L-US" device="L3225P" value="56nH"/>
-<part name="L8" library="rcl" deviceset="L-US" device="L3225P" value="39nH"/>
+<part name="L6" library="rcl" deviceset="L-US" device="L0805" value="68nH"/>
+<part name="L7" library="rcl" deviceset="L-US" device="L0805" value="56nH"/>
+<part name="L8" library="rcl" deviceset="L-US" device="L0805" value="39nH"/>
 <part name="C34" library="rcl" deviceset="C-EU" device="C0805" value="22pF"/>
 <part name="C35" library="rcl" deviceset="C-EU" device="C0805" value="33pF"/>
