File: circuit/cs4272_test.sch (EAGLE design)
At the start: 23 parts, among them IC1 CS4272

Commit message: - balmer.lbr CS4272 - STM32F405RGT6
Connections:
- removed net PA8: IC1.CCLK, SV1.10
- removed net PA9: IC1.CDIN, SV1.9
- new net CCLK: IC1.CCLK, SV1.9
- new net CDIN: IC1.CDIN, SV1.10
- net PA10: now also SV1.7; no longer SV1.8
- net PA13: now also SV1.8; no longer SV1.7
- net PA14: now also SV1.5; no longer SV1.6
- net PC11: now also SV1.4; no longer SV1.3
- net PD0: now also SV1.2; no longer SV1.1
- net SPI3_MOSI(PC12): now also SV1.1; no longer SV1.2
- net SPI3_NSS(PA15): now also SV1.6; no longer SV1.5
- net SPI3_SCK(PC10): now also SV1.3; no longer SV1.4
Other:
- moved on the sheet: SV1
Changed lines of the file:
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@@
 <part name="R8" library="rcl" deviceset="R-EU_" device="R0603" value="56"/>
 <part name="C1" library="rcl" deviceset="C-EU" device="C0805" value="10mk"/>
-<part name="SV1" library="con-ml" deviceset="ML10" device=""/>
 <part name="X1" library="con-phoenix-254" deviceset="MPT3" device=""/>
 <part name="GND6" library="supply1" deviceset="GND" device=""/>
@@
 <part name="C9" library="rcl" deviceset="C-EU" device="C0603" value="1mk"/>
 <part name="L1" library="rcl" deviceset="L-US" device="L0805" value="1000Z"/>
+<part name="SV1" library="con-ml" deviceset="ML10" device=""/>
 </parts>
 <sheets>
@@
 <instance part="R8" gate="G$1" x="40.64" y="53.34"/>
 <instance part="C1" gate="G$1" x="116.84" y="58.42"/>
-<instance part="SV1" gate="G$1" x="40.64" y="20.32" rot="MR180"/>
 <instance part="X1" gate="-1" x="144.78" y="43.18"/>
 <instance part="X1" gate="-2" x="144.78" y="38.1"/>
@@
 <instance part="C9" gate="G$1" x="121.92" y="73.66"/>
 <instance part="L1" gate="G$1" x="134.62" y="88.9" rot="R270"/>
+<instance part="SV1" gate="G$1" x="40.64" y="20.32" rot="R180"/>
 </instances>
 <busses>
@@
 </segment>
 <segment>
-<pinref part="SV1" gate="G$1" pin="5"/>
 <wire x1="48.26" y1="20.32" x2="58.42" y2="20.32" width="0.1524" layer="91"/>
 <label x="48.26" y="20.32" size="1.778" layer="95"/>
+<pinref part="SV1" gate="G$1" pin="6"/>
 </segment>
 </net>
@@
 </segment>
 <segment>
-<pinref part="SV1" gate="G$1" pin="4"/>
 <wire x1="33.02" y1="22.86" x2="25.4" y2="22.86" width="0.1524" layer="91"/>
 <label x="12.7" y="22.86" size="1.778" layer="95"/>
+<pinref part="SV1" gate="G$1" pin="3"/>
 </segment>
 </net>
@@
 </segment>
 <segment>
-<pinref part="SV1" gate="G$1" pin="2"/>
 <wire x1="33.02" y1="25.4" x2="25.4" y2="25.4" width="0.1524" layer="91"/>
 <label x="12.7" y="25.4" size="1.778" layer="95"/>
+<pinref part="SV1" gate="G$1" pin="1"/>
 </segment>
 </net>
@@
 <net name="PA14" class="0">
 <segment>
-<pinref part="SV1" gate="G$1" pin="6"/>
 <wire x1="33.02" y1="20.32" x2="25.4" y2="20.32" width="0.1524" layer="91"/>
 <label x="20.32" y="20.32" size="1.778" layer="95"/>
+<pinref part="SV1" gate="G$1" pin="5"/>
 </segment>
 </net>
 <net name="PA10" class="0">
 <segment>
-<pinref part="SV1" gate="G$1" pin="8"/>
 <wire x1="33.02" y1="17.78" x2="25.4" y2="17.78" width="0.1524" layer="91"/>
 <label x="20.32" y="17.78" size="1.778" layer="95"/>
+<pinref part="SV1" gate="G$1" pin="7"/>
 </segment>
 <segment>
@@
 <net name="PD0" class="0">
 <segment>
-<pinref part="SV1" gate="G$1" pin="1"/>
 <wire x1="48.26" y1="25.4" x2="58.42" y2="25.4" width="0.1524" layer="91"/>
 <label x="48.26" y="25.4" size="1.778" layer="95"/>
+<pinref part="SV1" gate="G$1" pin="2"/>
 </segment>
 <segment>
@@
 <net name="PC11" class="0">
 <segment>
-<pinref part="SV1" gate="G$1" pin="3"/>
 <wire x1="48.26" y1="22.86" x2="58.42" y2="22.86" width="0.1524" layer="91"/>
 <label x="48.26" y="22.86" size="1.778" layer="95"/>
+<pinref part="SV1" gate="G$1" pin="4"/>
 </segment>
 </net>
 <net name="PA13" class="0">
 <segment>
-<pinref part="SV1" gate="G$1" pin="7"/>
 <wire x1="48.26" y1="17.78" x2="58.42" y2="17.78" width="0.1524" layer="91"/>
 <label x="48.26" y="17.78" size="1.778" layer="95"/>
-</segment>
-</net>
-<net name="PA8" class="0">
-<segment>
-<pinref part="SV1" gate="G$1" pin="10"/>
+<pinref part="SV1" gate="G$1" pin="8"/>
+</segment>
+</net>
+<net name="CCLK" class="0">
+<segment>
 <wire x1="33.02" y1="15.24" x2="25.4" y2="15.24" width="0.1524" layer="91"/>
 <label x="20.32" y="15.24" size="1.778" layer="95"/>
+<pinref part="SV1" gate="G$1" pin="9"/>
 </segment>
 <segment>
@@
 </segment>
 </net>
-<net name="PA9" class="0">
-<segment>
-<pinref part="SV1" gate="G$1" pin="9"/>
+<net name="CDIN" class="0">
+<segment>
 <wire x1="48.26" y1="15.24" x2="58.42" y2="15.24" width="0.1524" layer="91"/>
 <label x="48.26" y="15.24" size="1.778" layer="95"/>
-</segment>
-<segment>
+<pinref part="SV1" gate="G$1" pin="10"/>
+</segment>
+<segment>
