File: circuit/ADC_DSP.brd (EAGLE design)
At the start: 100 x 80 mm, 49 parts, among them IC1 REG1117, IC2 AD8605, IC3 STM32F40XRXT6, IC4 CS4272, Q1 8MHz, Q2 24.576MHz

Commit message: - ??????? 51x57 ??
Parts:
- moved L2 29.2 mm to (10.2, 36.8), flipped to the bottom
- moved C25 28.2 mm to (31.1, 48.3)
- moved X4 27.5 mm to (24.8, 53.3)
- moved C26 27.3 mm to (19.1, 42.5), flipped to the bottom
- moved C20 26.5 mm to (19.1, 45.1)
- moved C22 26.1 mm to (19.1, 47.6)
- moved C23 24.3 mm to (35.6, 45.7)
- moved C24 24.3 mm to (35.6, 48.3)
- moved C18 24.3 mm to (39.4, 40.6)
- moved C19 24.3 mm to (39.4, 35.6)
- moved Q2 24.3 mm to (36.8, 38.1)
- moved R9 24.3 mm to (32.4, 34.3)
- moved C1 24.3 mm to (10.2, 15.9)
- moved C11 24.3 mm to (24.1, 14.0)
- moved C15 24.3 mm to (14.6, 29.2)
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Routing:
- net N$22: track 13.8 -> 9.70 mm, vias 2 -> 0
- net N$15: track 11.9 -> 8.16 mm
- net N$12: track 8.66 -> 12.3 mm
- net N$2: track 5.23 -> 8.40 mm
- net +3V3: track 107.3 -> 110.4 mm
- net N$16: track 11.1 -> 8.37 mm
- net N$17: track 11.8 -> 9.15 mm
- net N$23: track 7.61 -> 5.33 mm
- net N$14: track 32.5 -> 34.6 mm, vias 1 -> 2
- net N$20: track 6.40 -> 4.36 mm
- net N$18: track 12.6 -> 10.7 mm
- net GND: track 247.5 -> 245.6 mm, vias 3 -> 2
- net +5V: track 60.0 -> 58.8 mm, vias 3 -> 2
Other:
- board size 100 x 80 mm -> 50.5 x 57.1 mm

Commit message: - 43x55 ??
Parts:
- moved C17 7.10 mm to (21.0, 35.7)
- moved IC4 7.10 mm to (21.0, 41.3)
- moved C20 7.10 mm to (12.1, 43.8)
- moved C21 7.10 mm to (28.6, 49.5)
- moved C22 7.10 mm to (12.1, 46.4)
- moved C23 7.10 mm to (28.6, 44.5)
- moved C24 7.10 mm to (28.6, 47.0)
- moved C26 7.10 mm to (12.1, 41.3)
- moved C8 7.10 mm to (31.1, 24.8)
- moved IC2 7.10 mm to (30.5, 5.71)
- moved IC3 7.10 mm to (21.0, 21.6)
- moved C11 7.10 mm to (17.1, 12.7)
- moved C18 7.10 mm to (32.4, 39.4)
- moved C19 7.10 mm to (32.4, 34.3)
- moved Q1 7.10 mm to (10.2, 25.4)
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Routing:
- net GND: track 245.6 -> 238.0 mm
- net +3V3: track 110.4 -> 105.8 mm
- net V+: track 12.8 -> 8.49 mm
- net N$14: track 34.6 -> 31.5 mm, vias 2 -> 1
- net +5V: track 58.8 -> 60.5 mm
- net N$3: track 8.83 -> 7.16 mm
Other:
- board size 50.5 x 57.1 mm -> 43.5 x 55.2 mm

Commit message: - ???????? ???????????? (??????? ????? ? ?? ????? ???????)
Parts:
- added C27, C28, C29, C30: (no value), rcl:C0805
- added L3: (no value), rcl:L2012C
- moved X3 6.35 mm to (32.4, 9.53)
- moved R4 4.49 mm to (24.8, 8.89), turned to 0 degrees
- moved IC2 4.45 mm to (26.0, 5.71)
- moved R6 4.45 mm to (33.7, 3.17)
- moved R7 4.45 mm to (33.7, 5.08)
- moved C4 4.44 mm to (30.5, 4.45)
- moved R5 4.44 mm to (27.9, 9.53)
- moved R2 3.81 mm to (17.9, 7.87)
- moved C3 2.84 mm to (26.7, 12.7)
- moved C9 2.29 mm to (31.8, 19.7), turned to 90 degrees
- moved R1 2.01 mm to (23.2, 12.8), turned to 180 degrees
- moved X4 1.42 mm to (18.4, 50.8)
- moved C5 1.41 mm to (30.8, 14.6)
- moved C6 1.41 mm to (30.8, 16.9)
- moved X2 1.27 mm to (36.8, 22.9)
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Connections:
- net N$13 renamed VCOM
- net N$14 renamed AVCC
- new net AGND: C20.2, C21.2, C22.2, C23.2, C24.2, C25.2, C26.2, C27.2, C28.2, C29.2, C30.2, IC4.21, L3.2, X4.1
- net GND: now also L3.1; no longer C20.2, C21.2, C22.2, C23.2, C24.2, C25.2, C26.2, IC4.21, X4.1
- net N$15: now also C30.1
- net N$16: now also C29.1
- net N$17: now also C28.1
- net N$18: now also C27.1
Routing:
- net AGND: track 0.00 -> 69.3 mm, vias 0 -> 2
- net GND: track 238.0 -> 191.9 mm, vias 2 -> 3
- net +5V: track 60.5 -> 53.4 mm
- net N$24: track 4.20 -> 10.0 mm
- net +3V3: track 105.8 -> 101.4 mm
- net N$12: track 12.3 -> 14.8 mm
- net N$15: track 8.16 -> 10.6 mm
- net N$16: track 8.37 -> 10.3 mm
- net N$17: track 9.15 -> 11.1 mm
- net AVCC: track 31.5 -> 29.6 mm
- net N$21: track 3.26 -> 5.09 mm
- net N$7: track 10.6 -> 8.78 mm
- net VCOM: track 14.3 -> 12.6 mm
- net N$18: track 10.7 -> 11.9 mm
- net N$2: track 8.40 -> 9.33 mm
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Other:
- board size 43.5 x 55.2 mm -> 41.6 x 57.8 mm

Commit message: - ????? ? ?????????? GND ? AGND
Parts:
- moved C10 1.80 mm to (31.5, 26.0), turned to 0 degrees
- moved C8 1.35 mm to (31.5, 23.9), turned to 0 degrees
- moved X2 0.63 mm to (36.2, 22.9)
Routing:
- net N$28: track 0.00 -> 3.81 mm
- net N$26: track 0.00 -> 3.81 mm
- net N$29: track 0.00 -> 3.17 mm
- net N$14: track 0.00 -> 3.17 mm
- net N$27: track 0.00 -> 2.54 mm
- net N$25: track 0.00 -> 2.54 mm
- net N$30: track 0.00 -> 2.54 mm
- net N$13: track 0.00 -> 2.54 mm
- net GND: track 191.9 -> 190.6 mm
- net SWDCLK: track 17.6 -> 16.6 mm
- net SWDIO: track 12.4 -> 11.8 mm
- net +3V3: track 101.4 -> 100.8 mm
- added copper zone on layer 1, net AGND
- added copper zone on layer 16, net AGND
- added copper zone on layer 1, net GND
- added copper zone on layer 16, net GND
Other:
- board size 41.6 x 57.8 mm -> 40.3 x 57.8 mm
