File: circuit/ADC_DSP.brd (EAGLE design)
At the start: 40.3 x 57.8 mm, 54 parts, among them IC1 REG1117, IC2 AD8605, IC3 STM32F40XRXT6, IC4 CS4272, Q1 8MHz, Q2 24.576MHz

Commit message: - R3 3.3 KOm -> 33 KOm C2 10 nF -> 1 nF - ???????? ??? ??? ?? ????????? DAC
Parts:
- C2: value 10n -> 470
- R3: value 3.3k -> 33k
Changed lines of the file:
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@@
 <layer number="24" name="bOrigins" color="15" fill="1" visible="yes" active="yes"/>
 <layer number="25" name="tNames" color="7" fill="1" visible="yes" active="yes"/>
-<layer number="26" name="bNames" color="7" fill="1" visible="yes" active="yes"/>
+<layer number="26" name="bNames" color="7" fill="1" visible="no" active="yes"/>
 <layer number="27" name="tValues" color="7" fill="1" visible="no" active="yes"/>
 <layer number="28" name="bValues" color="7" fill="1" visible="no" active="yes"/>
@@
 <element name="C4" library="rcl" package="C0805" value="10u" x="30.48" y="4.445" rot="R270"/>
 <element name="C3" library="rcl" package="C0603" value="1u" x="26.67" y="12.7"/>
-<element name="C2" library="rcl" package="C0603" value="10n" x="17.145" y="10.16" rot="R180"/>
+<element name="C2" library="rcl" package="C0603" value="470" x="17.145" y="10.16" rot="R180"/>
 <element name="C7" library="rcl" package="C0603" value="100n" x="27.94" y="27.305"/>
 <element name="C12" library="rcl" package="C0603" value="100n" x="15.875" y="29.21" rot="R180"/>
@@
 <element name="R5" library="rcl" package="R0603" value="47k" x="27.94" y="9.525" rot="R90"/>
 <element name="R4" library="rcl" package="R0603" value="47k" x="24.765" y="8.89"/>
-<element name="R3" library="rcl" package="R0603" value="3.3k" x="20.32" y="12.7" rot="R90"/>
+<element name="R3" library="rcl" package="R0603" value="33k" x="20.32" y="12.7" rot="R90"/>
 <element name="X2" library="con-phoenix-254" package="4POL254" value="" x="36.195" y="22.86" rot="MR90">
 <attribute name="OC_NEWARK" value="unknown" x="36.195" y="22.86" size="1.778" layer="28" rot="MR90" display="off"/>

Commit message: - ?????????? ??????
Connections:
- net N$16 renamed AINB+
- net N$17 renamed AINA+
Changed lines of the file:
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@@
 <wire x1="20.955" y1="50.8" x2="20.955" y2="54.295" width="0.4064" layer="16"/>
 </signal>
-<signal name="N$16">
+<signal name="AINB+">
 <contactref element="IC4" pad="18"/>
 <contactref element="X4" pad="4"/>
@@
 <wire x1="18.415" y1="50.8" x2="18.415" y2="54.295" width="0.4064" layer="16"/>
 </signal>
-<signal name="N$17">
+<signal name="AINA+">
 <contactref element="IC4" pad="17"/>
 <contactref element="X4" pad="5"/>

Commit message: - ???????? ???????????? ADC_DSP.sch
Parts:
- removed C21, C23, C25: 10u, rcl:C0805
- removed IC2: AD8605, analog-devices:SOT23-5
- added SPI: (no value), con-phoenix-254:4POL254
- C1: value 10u -> 33uF; device rcl:C0805 -> rcl:153CLV-0605
- C10, C6: value 1u -> 2.2u
- C13: value 1u -> 0.1u
- C5: value 1u -> 220uF; device rcl:C0603 -> rcl:153CLV-0605
- C8: value 1u -> 33uF; device rcl:C0603 -> rcl:153CLV-0605
- R1: value 22k -> 56
- R2: value 4.7k -> 56
- R3: value 33k -> 22k
- R4, R5: value 47k -> 33
- R6: value 1k -> 33
- R7: value 10 -> 33
- moved C1 46.9 mm to (35.6, 52.1), turned to 270 degrees
- moved C8 38.6 mm to (5.08, 52.1), turned to 270 degrees
- moved R1 27.5 mm to (27.3, 40.0), flipped to the bottom, turned to 0 degrees
- moved C4 24.1 mm to (8.89, 15.2), turned to 90 degrees
- moved R2 19.4 mm to (9.53, 25.4)
- moved R6 15.9 mm to (32.4, 19.1)
- moved R7 15.9 mm to (32.4, 21.0)
- moved C5 13.7 mm to (21.0, 5.08), turned to 180 degrees
- moved R4 9.92 mm to (32.4, 15.2)
- moved R5 8.82 mm to (32.4, 17.1), turned to 0 degrees
- moved C6 6.87 mm to (25.1, 13.1)
- moved C9 5.85 mm to (27.9, 15.2), turned to 180 degrees
- moved X3 5.12 mm to (27.3, 8.89), turned to 270 degrees
- moved C3 4.58 mm to (22.9, 10.2)
- moved X2 3.86 mm to (36.8, 26.7)
Connections:
- new net N$16: C3.2, X3.1
- new net N$17: IC4.1, R1.2
- net +3V3: now also C5.+; no longer C1.1
- net +5V: no longer IC2.5, R4.1
- net AGND: now also C1.-, C8.-; no longer C21.2, C23.2, C25.2
- net AVCC: now also C8.+; no longer C25.1
- net GND: now also C4.2, C5.-; no longer C1.2, C5.2, C8.2, IC2.2, R2.2, R5.2, R6.2
- net N$1: no longer C8.1
- net N$12: now also C1.+; no longer C21.1, C23.1
- net N$19: now also IC3.6, R2.1; no longer C4.1, IC2.1, IC2.4
- net N$2: no longer C5.1
- net N$20: now also R4.2, SPI.1; no longer C4.2, R6.1, R7.1
- net N$21: now also R5.2, SPI.2; no longer R7.2, X3.1
- net N$22: now also R6.2, SPI.3; no longer C3.2, IC2.3, R4.2, R5.1
- net N$23: now also C3.1; no longer R1.2
- net N$24: now also R7.2, SPI.4; no longer C3.1, R1.1, R2.1
- net N$3: now also C4.1
- net N$6: now also R2.2; no longer IC3.6
- net N$8: now also R1.1; no longer IC4.1
- net SPI2_MISO: now also R6.1
- net SPI2_MOSI: now also R7.1
- net SPI2_NSS: now also R4.1
- net SPI2_SCK: now also R5.1
Routing:
- net +5V: track 53.4 -> 23.7 mm, vias 2 -> 0
- net GND: track 190.6 -> 163.3 mm, vias 3 -> 4
- net AGND: track 69.3 -> 91.7 mm
- net N$2: track 9.33 -> 2.86 mm
- net SPI2_NSS: track 0.00 -> 6.41 mm
- net SPI2_MOSI: track 0.00 -> 5.55 mm
- net SPI2_SCK: track 0.00 -> 5.37 mm
- net N$24: track 10.0 -> 4.65 mm
- net SPI2_MISO: track 0.00 -> 4.97 mm
- net +3V3: track 100.8 -> 96.3 mm
- net N$12: track 14.8 -> 18.8 mm, vias 0 -> 1
- net N$22: track 9.42 -> 5.50 mm
- net N$16: track 0.00 -> 3.59 mm
- net AVCC: track 29.6 -> 32.9 mm
- net SWDCLK: track 16.6 -> 13.4 mm
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
Commit message: - ?????? ?????????? ? ?????????????? ??????????????????
Connections:
- net +3V3: now also IC3.45
Routing:
- net +3V3: track 96.3 -> 108.9 mm
- net GND: track 163.3 -> 160.8 mm
Changed lines of the file:
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@@
 <setting verticaltext="up"/>
 </settings>
-<grid distance="0.635" unitdist="mm" unit="mm" style="lines" multiple="1" display="no" altdistance="0.25" altunitdist="mm" altunit="mm"/>
+<grid distance="0.635" unitdist="mm" unit="mm" style="lines" multiple="1" display="no" altdistance="0.125" altunitdist="mm" altunit="mm"/>
 <layers>
 <layer number="1" name="Top" color="4" fill="1" visible="yes" active="yes"/>
@@
 <wire x1="8.89" y1="16.19" x2="8.89" y2="16.51" width="0.4064" layer="1"/>
 <wire x1="8.89" y1="16.51" x2="7.7775" y2="17.6225" width="0.4064" layer="1"/>
-<wire x1="39.37" y1="30.48" x2="36.83" y2="30.48" width="0.6096" layer="1"/>
 <wire x1="29.845" y1="7.62" x2="27.305" y2="7.62" width="0.6096" layer="1"/>
 <wire x1="29.845" y1="7.62" x2="32.385" y2="7.62" width="0.6096" layer="1"/>
@@
 <wire x1="26.655" y1="25.34" x2="25.34" y2="25.34" width="0.25" layer="1"/>
 <wire x1="25.34" y1="25.34" x2="24.765" y2="24.765" width="0.25" layer="1"/>
-<wire x1="24.765" y1="24.765" x2="24.765" y2="18.415" width="0.25" layer="1"/>
+<wire x1="24.765" y1="24.765" x2="24.765" y2="24.13" width="0.25" layer="1"/>
+<wire x1="24.765" y1="24.13" x2="24.765" y2="23.495" width="0.25" layer="1"/>
+<wire x1="24.765" y1="23.495" x2="24.765" y2="18.415" width="0.25" layer="1"/>
 <wire x1="24.765" y1="18.415" x2="24.13" y2="17.78" width="0.25" layer="1"/>
 <wire x1="17.205" y1="27.29" x2="15.89" y2="27.29" width="0.25" layer="1"/>
@@
 <wire x1="26.67" y1="15.875" x2="26.67" y2="15.66" width="0.25" layer="1"/>
 <wire x1="26.67" y1="15.66" x2="27.09" y2="15.24" width="0.25" layer="1"/>
-<wire x1="28.575" y1="26.035" x2="36.83" y2="22.86" width="0" layer="19" extent="1-1"/>
+<wire x1="36.83" y1="22.86" x2="28.89" y2="22.86" width="0.25" layer="1"/>
+<contactref element="IC3" pad="45"/>
+<wire x1="26.655" y1="23.84" x2="25.055" y2="23.84" width="0.25" layer="1"/>
+<wire x1="25.055" y1="23.84" x2="24.765" y2="24.13" width="0.25" layer="1"/>
+<wire x1="26.655" y1="23.84" x2="27.91" y2="23.84" width="0.25" layer="1"/>
+<wire x1="27.91" y1="23.84" x2="28.89" y2="22.86" width="0.25" layer="1"/>
 </signal>
 <signal name="N$1">
