File: circuit/mixer.brd (EAGLE design)
At the start: 77.8 x 61 mm, 62 parts, among them IC1 74AC4053D, IC2 74AC74D, IC5 NE5534D, IC6 NE5534D, Q1 BFG135

Commit message: - ??? ????? ??????? ?????????
Parts:
- moved C38 9.85 mm to (62.5, 39.1), turned to 90 degrees
- moved C31 8.52 mm to (38.1, 34.9), turned to 90 degrees
- moved R18 8.03 mm to (56.5, 50.2), turned to 270 degrees
- moved R10 7.85 mm to (31.1, 40.6)
- moved R28 7.43 mm to (60.2, 39.0), turned to 270 degrees
- moved C18 7.33 mm to (45.7, 49.8)
- moved R27 7.10 mm to (60.3, 42.5), turned to 90 degrees
- moved R11 6.24 mm to (36.5, 39.1)
- moved R25 6.16 mm to (70.2, 53.3)
- moved R16 5.83 mm to (51.1, 55.9), turned to 90 degrees
- moved R20 5.79 mm to (49.5, 36.5)
- moved R21 5.62 mm to (51.1, 44.5), turned to 270 degrees
- moved C23 5.24 mm to (48.9, 55.9), turned to 270 degrees
- moved IC6 5.12 mm to (55.9, 38.7)
- moved C22 4.84 mm to (48.9, 44.5), turned to 90 degrees
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Connections:
- net +5V: no longer R18.2, R22.2
- net N$1: now also IC2.12, IC2.5; no longer IC2.2, IC2.9
- net N$2: now also IC2.2, IC2.8; no longer IC2.12, IC2.6
- net N$3: now also IC2.11, R6.2; no longer IC2.5, R10.1
- net N$31: now also IC2.9, R10.1; no longer IC2.3, R6.2
- net N$32: now also IC2.6, R11.1; no longer IC2.11, R7.2
- net N$4: now also IC2.3, R7.2; no longer IC2.8, R11.1
- net VDD: now also R18.2, R22.2
Routing:
- net GND: track 191.3 -> 237.9 mm, vias 2 -> 6
- net VDD: track 0.00 -> 46.0 mm
- net +5V: track 91.0 -> 115.3 mm, vias 0 -> 6
- net N$1: track 16.5 -> 7.20 mm, vias 2 -> 0
- net N$15: track 12.8 -> 21.2 mm
- net N$32: track 0.00 -> 8.28 mm
- net N$10: track 22.9 -> 15.1 mm
- net N$4: track 5.43 -> 13.0 mm
- net N$31: track 0.00 -> 6.67 mm
- net QOUTB: track 0.00 -> 5.67 mm
- net N$16: track 13.9 -> 9.12 mm
- net N$5: track 29.2 -> 24.6 mm
- net N$23: track 11.1 -> 14.8 mm
- net QOUT: track 0.00 -> 3.62 mm
- net N$17: track 14.8 -> 18.3 mm
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
Commit message: - ??????? ??? ????????
Parts:
- C6: value 100n -> 33n; device rcl:C0603 -> rcl:C0805
- moved L3 10.0 mm to (37.5, 20.0)
- moved C2 7.65 mm to (66.0, 44.5)
- moved R26 7.65 mm to (63.8, 44.5)
- moved R25 5.02 mm to (65.4, 51.8)
- moved C37 4.49 mm to (63.8, 49.5), turned to 0 degrees
- moved R24 4.49 mm to (64.5, 55.9)
- moved C1 4.32 mm to (67.0, 55.2)
- moved X2 3.18 mm to (20.9, 24.1)
- moved X3 3.18 mm to (41.4, 24.1)
- moved X4 3.18 mm to (10.8, 19.1)
- moved X5 2.54 mm to (71.8, 50.2)
- moved IC5 2.54 mm to (58.4, 52.7)
- moved R29 2.54 mm to (62.2, 52.7)
- moved R18 2.01 mm to (54.6, 50.8)
- moved C24 1.91 mm to (48.9, 50.2), turned to 270 degrees
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Routing:
- net N$30: track 0.00 -> 16.4 mm
- net N$29: track 0.00 -> 12.4 mm
- net N$27: track 0.00 -> 10.9 mm
- net VDD: track 46.0 -> 56.5 mm, vias 0 -> 2
- net GND: track 237.9 -> 248.3 mm
- net N$28: track 0.00 -> 7.66 mm
- net +5V: track 115.3 -> 119.3 mm
- net N$33: track 0.00 -> 3.48 mm
- net N$32: track 8.28 -> 5.86 mm
- net N$26: track 0.00 -> 2.31 mm
- net N$15: track 21.2 -> 19.1 mm
- net QOUTB: track 5.67 -> 3.63 mm
- net N$17: track 18.3 -> 16.2 mm
- net N$3: track 4.53 -> 3.59 mm
- net QOUT: track 3.62 -> 4.54 mm
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
Commit message: - ???????, ??????? ?????????
Parts:
- moved R20 10.6 mm to (43.8, 27.6)
- moved C1 10.6 mm to (61.3, 46.4)
- moved C14 10.6 mm to (34.9, 41.9)
- moved C15 10.6 mm to (29.8, 13.3)
- moved C16 10.6 mm to (27.3, 13.3)
- moved C2 10.6 mm to (60.3, 35.6)
- moved C22 10.6 mm to (43.2, 35.6)
- moved C23 10.6 mm to (43.2, 45.7)
- moved C24 10.6 mm to (43.2, 41.3)
- moved C32 10.6 mm to (48.3, 38.7)
- moved C37 10.6 mm to (58.1, 40.6)
- moved IC2 10.6 mm to (26.0, 24.1)
- moved IC5 10.6 mm to (52.7, 43.8)
- moved IC6 10.6 mm to (50.2, 29.8)
- moved L3 10.6 mm to (31.8, 11.1)
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Other:
- board size 77.8 x 61 mm -> 70.8 x 52.7 mm

Commit message: - ?????????? DDS ??????????. - ????????? ???????
Parts:
- R18, R19, R22, R23: value 22K -> 68K
