File: circuit/mixer.sch (EAGLE design)
At the start: 62 parts, among them IC1 74AC4053D, IC2 74AC74D, IC5 NE5534D, IC6 NE5534D, Q1 BFG135

Commit message: - ??? ????? ??????? ?????????
Connections:
- net +5V: no longer R18.2, R22.2
- net N$1: now also IC2A.Q, IC2B.D; no longer IC2A.D, IC2B.Q
- net N$2: now also IC2A.D, IC2B.!Q; no longer IC2A.!Q, IC2B.D
- net N$3: now also IC2B.CLK, R6.2; no longer IC2A.Q, R10.1
- net N$31: now also IC2B.Q, R10.1; no longer IC2A.CLK, R6.2
- net N$32: now also IC2A.!Q, R11.1; no longer IC2B.CLK, R7.2
- net N$4: now also IC2A.CLK, R7.2; no longer IC2B.!Q, R11.1
- net VDD: now also R18.2, R22.2
Other:
- moved on the sheet: IC2A, IC2B, R18, R19, R22, R23
Changed lines of the file:
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@@
 <part name="R23" library="rcl" deviceset="R-EU_" device="R0603" value="22K"/>
 <part name="GND9" library="supply1" deviceset="GND" device=""/>
-<part name="P+6" library="supply1" deviceset="+5V" device=""/>
 <part name="R18" library="rcl" deviceset="R-EU_" device="R0603" value="22K"/>
 <part name="R19" library="rcl" deviceset="R-EU_" device="R0603" value="22K"/>
@@
 <part name="R16" library="rcl" deviceset="R-EU_" device="R0603" value="1K"/>
 <part name="R17" library="rcl" deviceset="R-EU_" device="R0603" value="1K"/>
-<part name="P+8" library="supply1" deviceset="+5V" device=""/>
 <part name="GND18" library="supply1" deviceset="GND" device=""/>
 <part name="P+9" library="supply1" deviceset="VCC" device=""/>
@@
 <part name="VDD2" library="supply1" deviceset="VDD" device=""/>
 <part name="VDD3" library="supply1" deviceset="VDD" device=""/>
+<part name="VDD4" library="supply1" deviceset="VDD" device=""/>
+<part name="VDD5" library="supply1" deviceset="VDD" device=""/>
 </parts>
 <sheets>
@@
 <instance part="IC1" gate="A" x="35.56" y="63.5" rot="MR0"/>
 <instance part="IC1" gate="P" x="83.82" y="-7.62"/>
-<instance part="IC2" gate="A" x="35.56" y="17.78"/>
-<instance part="IC2" gate="B" x="35.56" y="-5.08"/>
+<instance part="IC2" gate="A" x="35.56" y="-5.08"/>
+<instance part="IC2" gate="B" x="35.56" y="17.78"/>
 <instance part="IC2" gate="P" x="93.98" y="-7.62"/>
 <instance part="P+1" gate="1" x="17.78" y="27.94"/>
@@
 <instance part="R28" gate="G$1" x="139.7" y="22.86"/>
 <instance part="R29" gate="G$1" x="137.16" y="73.66"/>
-<instance part="R22" gate="G$1" x="101.6" y="30.48" rot="R90"/>
-<instance part="R23" gate="G$1" x="101.6" y="20.32" rot="R90"/>
-<instance part="GND9" gate="1" x="101.6" y="12.7"/>
-<instance part="P+6" gate="1" x="101.6" y="38.1"/>
-<instance part="R18" gate="G$1" x="101.6" y="76.2" rot="R90"/>
-<instance part="R19" gate="G$1" x="101.6" y="66.04" rot="R90"/>
-<instance part="GND10" gate="1" x="101.6" y="58.42"/>
+<instance part="R22" gate="G$1" x="101.6" y="27.94" rot="R90"/>
+<instance part="R23" gate="G$1" x="101.6" y="17.78" rot="R90"/>
+<instance part="GND9" gate="1" x="101.6" y="10.16"/>
+<instance part="R18" gate="G$1" x="101.6" y="73.66" rot="R90"/>
+<instance part="R19" gate="G$1" x="101.6" y="63.5" rot="R90"/>
+<instance part="GND10" gate="1" x="101.6" y="55.88"/>
 <instance part="C38" gate="G$1" x="149.86" y="43.18" rot="R90"/>
 <instance part="C37" gate="G$1" x="149.86" y="91.44" rot="R90"/>
@@
 <instance part="R16" gate="G$1" x="101.6" y="93.98"/>
 <instance part="R17" gate="G$1" x="101.6" y="86.36"/>
-<instance part="P+8" gate="1" x="101.6" y="83.82"/>
 <instance part="GND18" gate="1" x="83.82" y="-45.72"/>
 <instance part="P+9" gate="VCC" x="93.98" y="-30.48"/>
@@
 <instance part="VDD2" gate="G$1" x="132.08" y="53.34"/>
 <instance part="VDD3" gate="G$1" x="129.54" y="104.14"/>
+<instance part="VDD4" gate="G$1" x="101.6" y="81.28"/>
+<instance part="VDD5" gate="G$1" x="101.6" y="35.56"/>
 </instances>
 <busses>
@@
 <net name="+5V" class="0">
 <segment>
+<pinref part="P+1" gate="1" pin="+5V"/>
+<wire x1="17.78" y1="22.86" x2="17.78" y2="25.4" width="0.1524" layer="91"/>
+<wire x1="17.78" y1="12.7" x2="17.78" y2="22.86" width="0.1524" layer="91"/>
+<wire x1="17.78" y1="0" x2="17.78" y2="12.7" width="0.1524" layer="91"/>
+<wire x1="17.78" y1="-10.16" x2="17.78" y2="0" width="0.1524" layer="91"/>
+<pinref part="IC2" gate="B" pin="PRE"/>
+<wire x1="22.86" y1="22.86" x2="17.78" y2="22.86" width="0.1524" layer="91"/>
+<pinref part="IC2" gate="A" pin="CLR"/>
+<wire x1="22.86" y1="-10.16" x2="17.78" y2="-10.16" width="0.1524" layer="91"/>
 <pinref part="IC2" gate="A" pin="PRE"/>
-<pinref part="P+1" gate="1" pin="+5V"/>
-<wire x1="22.86" y1="22.86" x2="17.78" y2="22.86" width="0.1524" layer="91"/>
-<wire x1="17.78" y1="22.86" x2="17.78" y2="25.4" width="0.1524" layer="91"/>
-<pinref part="IC2" gate="A" pin="CLR"/>
+<wire x1="22.86" y1="0" x2="17.78" y2="0" width="0.1524" layer="91"/>
+<pinref part="IC2" gate="B" pin="CLR"/>
 <wire x1="22.86" y1="12.7" x2="17.78" y2="12.7" width="0.1524" layer="91"/>
-<wire x1="17.78" y1="12.7" x2="17.78" y2="22.86" width="0.1524" layer="91"/>
-<pinref part="IC2" gate="B" pin="PRE"/>
-<wire x1="22.86" y1="0" x2="17.78" y2="0" width="0.1524" layer="91"/>
-<wire x1="17.78" y1="0" x2="17.78" y2="12.7" width="0.1524" layer="91"/>
-<pinref part="IC2" gate="B" pin="CLR"/>
-<wire x1="22.86" y1="-10.16" x2="17.78" y2="-10.16" width="0.1524" layer="91"/>
-<wire x1="17.78" y1="-10.16" x2="17.78" y2="0" width="0.1524" layer="91"/>
 <junction x="17.78" y="0"/>
 <junction x="17.78" y="12.7"/>
@@
 <pinref part="P+4" gate="1" pin="+5V"/>
 <wire x1="17.78" y1="83.82" x2="17.78" y2="86.36" width="0.1524" layer="91"/>
-</segment>
-<segment>
-<pinref part="R22" gate="G$1" pin="2"/>
-<pinref part="P+6" gate="1" pin="+5V"/>
-</segment>
-<segment>
-<pinref part="R18" gate="G$1" pin="2"/>
-<pinref part="P+8" gate="1" pin="+5V"/>
 </segment>
 <segment>
@@
 <net name="N$1" class="0">
 <segment>
-<pinref part="IC2" gate="A" pin="D"/>
-<wire x1="22.86" y1="20.32" x2="20.32" y2="20.32" width="0.1524" layer="91"/>
 <wire x1="20.32" y1="20.32" x2="20.32" y2="7.62" width="0.1524" layer="91"/>
-<pinref part="IC2" gate="B" pin="Q"/>
 <wire x1="20.32" y1="7.62" x2="48.26" y2="7.62" width="0.1524" layer="91"/>
+<pinref part="IC2" gate="A" pin="Q"/>
 <wire x1="48.26" y1="7.62" x2="48.26" y2="0" width="0.1524" layer="91"/>
+<pinref part="IC2" gate="B" pin="D"/>
+<wire x1="20.32" y1="20.32" x2="22.86" y2="20.32" width="0.1524" layer="91"/>
 </segment>
 </net>
 <net name="N$2" class="0">
 <segment>
-<pinref part="IC2" gate="B" pin="D"/>
-<wire x1="22.86" y1="-2.54" x2="20.32" y2="-2.54" width="0.1524" layer="91"/>
 <wire x1="20.32" y1="-2.54" x2="20.32" y2="5.08" width="0.1524" layer="91"/>
 <wire x1="20.32" y1="5.08" x2="50.8" y2="5.08" width="0.1524" layer="91"/>
 <wire x1="50.8" y1="5.08" x2="50.8" y2="12.7" width="0.1524" layer="91"/>
-<pinref part="IC2" gate="A" pin="!Q"/>
+<pinref part="IC2" gate="A" pin="D"/>
+<wire x1="20.32" y1="-2.54" x2="22.86" y2="-2.54" width="0.1524" layer="91"/>
+<pinref part="IC2" gate="B" pin="!Q"/>
 <wire x1="50.8" y1="12.7" x2="48.26" y2="12.7" width="0.1524" layer="91"/>
-</segment>
-</net>
-<net name="N$3" class="0">
-<segment>
-<pinref part="IC2" gate="A" pin="Q"/>
-<pinref part="R10" gate="G$1" pin="1"/>
-<wire x1="48.26" y1="22.86" x2="50.8" y2="22.86" width="0.1524" layer="91"/>
-</segment>
-</net>
-<net name="N$4" class="0">
-<segment>
-<pinref part="IC2" gate="B" pin="!Q"/>
-<pinref part="R11" gate="G$1" pin="1"/>
-<wire x1="48.26" y1="-10.16" x2="50.8" y2="-10.16" width="0.1524" layer="91"/>
 </segment>
 </net>
@@
 <wire x1="119.38" y1="40.64" x2="109.22" y2="40.64" width="0.1524" layer="91"/>
 <wire x1="109.22" y1="40.64" x2="106.68" y2="40.64" width="0.1524" layer="91"/>
-<wire x1="101.6" y1="25.4" x2="109.22" y2="25.4" width="0.1524" layer="91"/>
-<wire x1="109.22" y1="25.4" x2="109.22" y2="40.64" width="0.1524" layer="91"/>
+<wire x1="101.6" y1="22.86" x2="109.22" y2="22.86" width="0.1524" layer="91"/>
+<wire x1="109.22" y1="22.86" x2="109.22" y2="40.64" width="0.1524" layer="91"/>
 <junction x="109.22" y="40.64"/>
-<junction x="101.6" y="25.4"/>
+<junction x="101.6" y="22.86"/>
 </segment>
 </net>
@@
 <wire x1="116.84" y1="88.9" x2="109.22" y2="88.9" width="0.1524" layer="91"/>
 <wire x1="109.22" y1="88.9" x2="109.22" y2="86.36" width="0.1524" layer="91"/>
-<wire x1="101.6" y1="71.12" x2="109.22" y2="71.12" width="0.1524" layer="91"/>
-<wire x1="109.22" y1="71.12" x2="109.22" y2="86.36" width="0.1524" layer="91"/>
-<junction x="101.6" y="71.12"/>
+<wire x1="101.6" y1="68.58" x2="109.22" y2="68.58" width="0.1524" layer="91"/>
+<wire x1="109.22" y1="68.58" x2="109.22" y2="86.36" width="0.1524" layer="91"/>
+<junction x="101.6" y="68.58"/>
 <junction x="109.22" y="86.36"/>
 </segment>
@@
 </segment>
 </net>
-<net name="N$31" class="0">
-<segment>
-<pinref part="IC2" gate="A" pin="CLK"/>
-<wire x1="22.86" y1="15.24" x2="12.7" y2="15.24" width="0.1524" layer="91"/>
-<pinref part="R6" gate="G$1" pin="2"/>
-</segment>
-</net>
 <net name="QOUTB" class="0">
 <segment>
@@
 <wire x1="-71.12" y1="-7.62" x2="-81.28" y2="-7.62" width="0.1524" layer="91"/>
 <label x="-84.074" y="-7.112" size="1.778" layer="95"/>
-</segment>
-</net>
-<net name="N$32" class="0">
-<segment>
-<pinref part="IC2" gate="B" pin="CLK"/>
-<wire x1="22.86" y1="-7.62" x2="12.7" y2="-7.62" width="0.1524" layer="91"/>
-<pinref part="R7" gate="G$1" pin="2"/>
 </segment>
 </net>
@@
 <pinref part="C2" gate="G$1" pin="1"/>
 <wire x1="175.26" y1="68.58" x2="180.34" y2="68.58" width="0.1524" layer="91"/>
+<junction x="180.34" y="68.58"/>
 </segment>
 </net>
@@
 <junction x="129.54" y="101.6"/>
 </segment>
-</net>
+<segment>
+<pinref part="R18" gate="G$1" pin="2"/>
+<pinref part="VDD4" gate="G$1" pin="VDD"/>
+</segment>
+<segment>
+<pinref part="R22" gate="G$1" pin="2"/>
+<pinref part="VDD5" gate="G$1" pin="VDD"/>
+</segment>
+</net>
+<net name="N$3" class="0">
+<segment>
+<pinref part="IC2" gate="B" pin="CLK"/>
+<pinref part="R6" gate="G$1" pin="2"/>
+<wire x1="22.86" y1="15.24" x2="12.7" y2="15.24" width="0.1524" layer="91"/>
+</segment>
+</net>
+<net name="N$4" class="0">
+<segment>
+<pinref part="IC2" gate="A" pin="CLK"/>
+<pinref part="R7" gate="G$1" pin="2"/>
+<wire x1="22.86" y1="-7.62" x2="12.7" y2="-7.62" width="0.1524" layer="91"/>
+</segment>
+</net>
+<net name="N$31" class="0">
+<segment>
+<pinref part="IC2" gate="B" pin="Q"/>
+<pinref part="R10" gate="G$1" pin="1"/>
+<wire x1="48.26" y1="22.86" x2="50.8" y2="22.86" width="0.1524" layer="91"/>
+</segment>
+</net>
+<net name="N$32" class="0">
+<segment>
+<pinref part="IC2" gate="A" pin="!Q"/>
+<pinref part="R11" gate="G$1" pin="1"/>
+<wire x1="48.26" y1="-10.16" x2="50.8" y2="-10.16" width="0.1524" layer="91"/>
+</segment>
+</net>

Commit message: - ??????? ??? ????????
Parts:
- C6: value 100n -> 33n; device rcl:C-EUC0603 -> rcl:C-EUC0805
Changed lines of the file:
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@@
 <part name="GND21" library="supply1" deviceset="GND" device=""/>
 <part name="GND22" library="supply1" deviceset="GND" device=""/>
-<part name="C6" library="rcl" deviceset="C-EU" device="C0603" value="100n"/>
+<part name="C6" library="rcl" deviceset="C-EU" device="C0805" value="33n"/>
 <part name="C14" library="rcl" deviceset="C-EU" device="C0603" value="100n"/>
 <part name="GND23" library="supply1" deviceset="GND" device=""/>

Commit message: - ?????????? DDS ??????????. - ????????? ???????
Parts:
- R18, R19, R22, R23: value 22K -> 68K
Changed lines of the file:
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@@
 <part name="R28" library="rcl" deviceset="R-EU_" device="R0603" value="10K"/>
 <part name="R29" library="rcl" deviceset="R-EU_" device="R0603" value="10K"/>
-<part name="R22" library="rcl" deviceset="R-EU_" device="R0603" value="22K"/>
-<part name="R23" library="rcl" deviceset="R-EU_" device="R0603" value="22K"/>
+<part name="R22" library="rcl" deviceset="R-EU_" device="R0603" value="68K"/>
+<part name="R23" library="rcl" deviceset="R-EU_" device="R0603" value="68K"/>
 <part name="GND9" library="supply1" deviceset="GND" device=""/>
-<part name="R18" library="rcl" deviceset="R-EU_" device="R0603" value="22K"/>
-<part name="R19" library="rcl" deviceset="R-EU_" device="R0603" value="22K"/>
+<part name="R18" library="rcl" deviceset="R-EU_" device="R0603" value="68K"/>
+<part name="R19" library="rcl" deviceset="R-EU_" device="R0603" value="68K"/>
 <part name="GND10" library="supply1" deviceset="GND" device=""/>
 <part name="C38" library="rcl" deviceset="C-EU" device="C0805" value="10mk"/>
