File: circuit/ADC_DSP.sch (EAGLE design)
At the start: 27 parts, among them IC1 STM32F40XRXT6, IC2 REG1117, IC3 CS4272, Q1 8MHz, Q2 24.576MHz

Commit message: - ?????? ????? ????????? ?????
Parts:
- added C17, C19, C22, C24: 10u, rcl:C-EUC0805
- added C18: 47n, rcl:C-EUC0805
- added C20, C23, C25: 1u, rcl:C-EUC0603
- added C21: 100n, rcl:C-EUC0603
- added C26: 10n, rcl:C-EUC0603
- added IC4: AD8605, analog-devices:AD8603UJ
- added IN: (no value), con-phoenix-254:MPT7
- added L2: 100u, rcl:L-US0207/12
- added PHONE: (no value), con-phoenix-254:MPT2
- added R10: 22k, rcl:R-EU_R0603
- added R11: 4.7k, rcl:R-EU_R0603
- added R5: 1k, rcl:R-EU_R0603
- added R6: 10, rcl:R-EU_R0603
- added R7, R8: 47k, rcl:R-EU_R0603
- added R9: 3.3k, rcl:R-EU_R0603
- added SWD: (no value), con-phoenix-254:MPT4
Connections:
- new net +5V: IC4.+VS, L2.1, R8.1, X1-3.1
- new net DAC_OUT1: IC1PORTA_L.PA4, R9.2
- new net N$12: C17.1, C18.1, C19.1, IC3.FILT+
- new net N$13: C20.1, C21.1, IC3.VCOM, IN-7.1
- new net N$14: C22.1, C23.1, IC3.VA, IN-2.1, L2.2
- new net N$15: IC3.AINB-, IN-3.1
- new net N$16: IC3.AINB+, IN-4.1
- new net N$17: IC3.AINA+, IN-5.1
- new net N$18: IC3.AINA-, IN-6.1
- new net N$19: C24.1, IC4.IN-, IC4.OUT
- new net N$20: C24.2, R5.1, R6.1
- new net N$21: PHONE-1.1, R6.2
- new net N$22: C25.2, IC4.IN+, R7.1, R8.2
- new net N$23: C26.1, R10.2, R9.1
- new net N$24: C25.1, R10.1, R11.1
- new net SPI2_MISO: IC1PORTB_H.PB14
- new net SPI2_MOSI: IC1PORTB_H.PB15
- new net SPI2_NSS: IC1PORTB_H.PB12
- new net SPI2_SCK: IC1PORTB_H.PB13
- net +3V3: now also SWD-1.1; no longer X1-1.1
- net GND: now also C17.2, C18.2, C19.2, C20.2, C21.2, C22.2, C23.2, C26.2, IC3.AGND, IC4.-VS, IN-1.1, PHONE-2.1, R11.2, R5.2, R7.2, SWD-4.1
- net PB6: now also IC1PORTB_L.PB6
- net PB7: now also IC1PORTB_L.PB7
- net PB8: now also IC1PORTB_H.PB8
- net SWDCLK: now also SWD-3.1; no longer X1-3.1
- net SWDIO: now also SWD-2.1; no longer X1-2.1
- net V+: now also X1-1.1, X1-2.1
Other:
- moved on the sheet: X1-1, X1-2, X1-3, X1-4

Commit message: - ?????? ???????????????? ??????
Parts:
- C1, C21, C4: value 100n -> 10u; device rcl:C-EUC0603 -> rcl:C-EUC0805
- C10, C3: value 100n -> 1u
- C11, C12, C14: value 22p -> 100n
- C13, C17: value 10u -> 1u; device rcl:C-EUC0805 -> rcl:C-EUC0603
- C16: value 1u -> 22p
- C18: value 47n -> 22p; device rcl:C-EUC0805 -> rcl:C-EUC0603
- C19: value 10u -> 22p; device rcl:C-EUC0805 -> rcl:C-EUC0603
- C2: value 100n -> 10n
- C22: value 10u -> 100n; device rcl:C-EUC0805 -> rcl:C-EUC0603
- C23, C25: value 1u -> 10u; device rcl:C-EUC0603 -> rcl:C-EUC0805
- C24: value 10u -> 47n
- C26: value 10n -> 1u
- C7, C9: value 1u -> 100n
- IC1: value STM32F40XRXT6 -> REG1117; device stm32:STM32F40XRXT6 -> burr-brown:REG1117
- IC2: value REG1117 -> AD8605; device burr-brown:REG1117 -> analog-devices:AD8603UJ
- IC3: value CS4272 -> STM32F40XRXT6; device balmer:CS4272 -> stm32:STM32F40XRXT6
- IC4: value AD8605 -> CS4272; device analog-devices:AD8603UJ -> balmer:CS4272
- R1: value 56 -> 22k
- R10: value 22k -> 56
- R11: value 4.7k -> 56
- R2: value 56 -> 4.7k
- R3: value 56 -> 3.3k
- R4: value 4.7k -> 47k
- R5: value 1k -> 47k
- R6: value 10 -> 1k
- R7: value 47k -> 10
- R8: value 47k -> 4.7k
- R9: value 3.3k -> 56
- renumbered IN to X4, PHONE to X3, SWD to X2
Connections:
- net +3V3: now also C1.1, C11.2, C12.2, C17.2, C7.2, C9.2, IC1.VOUT, IC3POWER.VBAT, IC3POWER.VDD1, IC3POWER.VDD2, IC3POWER.VDD3, IC3POWER.VDD4, IC4.VD, IC4.VL, R8.1; no longer C1.2, C13.1, C16.2, C2.2, C3.2, C4.2, IC1POWER.VBAT, IC1POWER.VDD1, IC1POWER.VDD2, IC1POWER.VDD3, IC1POWER.VDD4, IC2.VOUT, IC3.VD, IC3.VL, R4.1
- net +5V: now also IC2.+VS, R4.1; no longer IC4.+VS, R8.1
- net DAC_OUT1: now also IC3PORTA_L.PA4, R3.2; no longer IC1PORTA_L.PA4, R9.2
- net GND: now also C1.2, C11.1, C12.1, C14.2, C15.2, C16.2, C17.1, C18.1, C19.1, C2.2, C24.2, C25.2, C7.1, C9.1, IC1.GND, IC2.-VS, IC3BOOT_RST.BOOT0, IC3POWER.VSS1, IC3POWER.VSS2, IC3POWER.VSSA, IC4.AGND, IC4.CS_, IC4.DGND, R2.2, R6.2; no longer C1.1, C11.2, C12.2, C14.1, C15.1, C16.1, C17.2, C18.2, C19.2, C2.1, C3.1, C4.1, C7.2, C9.2, IC1BOOT_RST.BOOT0, IC1POWER.VSS1, IC1POWER.VSS2, IC1POWER.VSSA, IC2.GND, IC3.AGND, IC3.CS_, IC3.DGND, IC4.-VS, R11.2, R7.2
- net N$1: now also C10.1, C8.1, IC3POWER.VCAP2; no longer C5.1, C6.1, IC1POWER.VCAP2
- net N$10: now also IC4.SCLK, R9.2; no longer IC3.SCLK, R2.2
- net N$11: now also IC4.SDOUT, R10.2; no longer IC3.SDOUT, R3.2
- net N$12: now also C21.1, C23.1, C24.1, IC4.FILT+; no longer C17.1, C18.1, C19.1, IC3.FILT+
- net N$13: now also C22.1, IC4.VCOM; no longer C21.1, IC3.VCOM
- net N$14: now also C25.1, C26.1, IC4.VA; no longer C22.1, C23.1, IC3.VA
- net N$15: now also IC4.AINB-; no longer IC3.AINB-
- net N$16: now also IC4.AINB+; no longer IC3.AINB+
- net N$17: now also IC4.AINA+; no longer IC3.AINA+
- net N$18: now also IC4.AINA-; no longer IC3.AINA-
- net N$19: now also C4.1, IC2.IN-, IC2.OUT; no longer C24.1, IC4.IN-, IC4.OUT
- net N$2: now also C5.1, C6.1, IC3POWER.VCAP1; no longer C7.1, C8.1, IC1POWER.VCAP1
- net N$20: now also C4.2, R7.1; no longer C24.2, R5.1
- net N$21: now also R7.2; no longer R6.2
- net N$22: now also C3.2, IC2.IN+, R4.2, R5.1; no longer C25.2, IC4.IN+, R7.1, R8.2
- net N$23: now also C2.1, R1.2, R3.1; no longer C26.1, R10.2, R9.1
- net N$24: now also C3.1, R1.1, R2.1; no longer C25.1, R10.1, R11.1
- net N$3: now also C13.1, IC3POWER.VDDA; no longer C9.1, IC1POWER.VDDA
- net N$4: now also C14.1, IC3BOOT_RST.NRST; no longer C10.1, IC1BOOT_RST.NRST
- net N$5: now also C15.1, IC3OSC.OSC_IN; no longer C11.1, IC1OSC.OSC_IN
- net N$6: now also C16.1, IC3OSC.OSC_OUT; no longer C12.1, IC1OSC.OSC_OUT
- net N$7: now also C19.2, IC4.XTI; no longer C15.2, IC3.XTI
- net N$8: now also C18.2, IC4.XTO; no longer C14.2, IC3.XTO
- net N$9: now also IC4.LRCK, R11.2; no longer IC3.LRCK, R1.2
- net PA15(SPI3_NSS): now also IC3PORTA_H.PA15, R11.1; no longer IC1PORTA_H.PA15, R1.1
- net PB6: now also IC3PORTB_L.PB6, IC4.CCLK; no longer IC1PORTB_L.PB6, IC3.CCLK
- net PB7: now also IC3PORTB_L.PB7, IC4.CDIN, R8.2; no longer IC1PORTB_L.PB7, IC3.CDIN, R4.2
- net PB8: now also IC3PORTB_H.PB8, IC4.RST_; no longer IC1PORTB_H.PB8, IC3.RST_
- net PC10(SPI3_SCK): now also IC3PORTC_H.PC10, R9.1; no longer IC1PORTC_H.PC10, R2.1
- net PC12(I2S3_SD): now also IC3PORTC_H.PC12, R10.1; no longer IC1PORTC_H.PC12, R3.1
- net SPI2_MISO: now also IC3PORTB_H.PB14; no longer IC1PORTB_H.PB14
- net SPI2_MOSI: now also IC3PORTB_H.PB15; no longer IC1PORTB_H.PB15
- net SPI2_NSS: now also IC3PORTB_H.PB12; no longer IC1PORTB_H.PB12
- net SPI2_SCK: now also IC3PORTB_H.PB13; no longer IC1PORTB_H.PB13
- net SWDCLK: now also IC3PORTA_H.PA14; no longer IC1PORTA_H.PA14
- net SWDIO: now also IC3PORTA_H.PA13; no longer IC1PORTA_H.PA13
- net V+: now also IC1.VIN; no longer IC2.VIN
Other:
- moved on the sheet: C1, C10, C11, C12, C13, C14, C15, C16, C17, C18, C19, C2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

Commit message: - ???????? ???????????? (??????? ????? ? ?? ????? ???????)
Parts:
- added C27, C28, C29, C30: (no value), rcl:C-EUC0805
- added L3: (no value), rcl:L-USL2012C
Connections:
- net N$13 renamed VCOM
- net N$14 renamed AVCC
- new net AGND: C20.2, C21.2, C22.2, C23.2, C24.2, C25.2, C26.2, C27.2, C28.2, C29.2, C30.2, IC4.AGND, L3.2, X4-1.1
- net GND: now also L3.1; no longer C20.2, C21.2, C22.2, C23.2, C24.2, C25.2, C26.2, IC4.AGND, X4-1.1
- net N$15: now also C30.1
- net N$16: now also C29.1
- net N$17: now also C28.1
- net N$18: now also C27.1

Commit message: - R3 3.3 KOm -> 33 KOm C2 10 nF -> 1 nF - ???????? ??? ??? ?? ????????? DAC
Parts:
- C2: value 10n -> 470
- R3: value 3.3k -> 33k
Changed lines of the file:
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@@
 <grid distance="0.1" unitdist="inch" unit="inch" style="lines" multiple="1" display="no" altdistance="0.01" altunitdist="inch" altunit="inch"/>
 <layers>
-<layer number="1" name="Top" color="4" fill="1" visible="yes" active="no"/>
-<layer number="16" name="Bottom" color="1" fill="1" visible="yes" active="no"/>
-<layer number="17" name="Pads" color="2" fill="1" visible="yes" active="no"/>
-<layer number="18" name="Vias" color="2" fill="1" visible="yes" active="no"/>
-<layer number="19" name="Unrouted" color="6" fill="1" visible="yes" active="no"/>
-<layer number="20" name="Dimension" color="15" fill="1" visible="yes" active="no"/>
-<layer number="21" name="tPlace" color="7" fill="1" visible="yes" active="no"/>
-<layer number="22" name="bPlace" color="7" fill="1" visible="yes" active="no"/>
-<layer number="23" name="tOrigins" color="15" fill="1" visible="yes" active="no"/>
-<layer number="24" name="bOrigins" color="15" fill="1" visible="yes" active="no"/>
-<layer number="25" name="tNames" color="7" fill="1" visible="yes" active="no"/>
-<layer number="26" name="bNames" color="7" fill="1" visible="yes" active="no"/>
-<layer number="27" name="tValues" color="7" fill="1" visible="yes" active="no"/>
-<layer number="28" name="bValues" color="7" fill="1" visible="yes" active="no"/>
+<layer number="1" name="Top" color="4" fill="1" visible="no" active="no"/>
+<layer number="16" name="Bottom" color="1" fill="1" visible="no" active="no"/>
+<layer number="17" name="Pads" color="2" fill="1" visible="no" active="no"/>
+<layer number="18" name="Vias" color="2" fill="1" visible="no" active="no"/>
+<layer number="19" name="Unrouted" color="6" fill="1" visible="no" active="no"/>
+<layer number="20" name="Dimension" color="15" fill="1" visible="no" active="no"/>
+<layer number="21" name="tPlace" color="7" fill="1" visible="no" active="no"/>
+<layer number="22" name="bPlace" color="7" fill="1" visible="no" active="no"/>
+<layer number="23" name="tOrigins" color="15" fill="1" visible="no" active="no"/>
+<layer number="24" name="bOrigins" color="15" fill="1" visible="no" active="no"/>
+<layer number="25" name="tNames" color="7" fill="1" visible="no" active="no"/>
+<layer number="26" name="bNames" color="7" fill="1" visible="no" active="no"/>
+<layer number="27" name="tValues" color="7" fill="1" visible="no" active="no"/>
+<layer number="28" name="bValues" color="7" fill="1" visible="no" active="no"/>
 <layer number="29" name="tStop" color="7" fill="3" visible="no" active="no"/>
 <layer number="30" name="bStop" color="7" fill="6" visible="no" active="no"/>
@@
 <layer number="35" name="tGlue" color="7" fill="4" visible="no" active="no"/>
 <layer number="36" name="bGlue" color="7" fill="5" visible="no" active="no"/>
-<layer number="37" name="tTest" color="7" fill="1" visible="yes" active="no"/>
-<layer number="38" name="bTest" color="7" fill="1" visible="yes" active="no"/>
+<layer number="37" name="tTest" color="7" fill="1" visible="no" active="no"/>
+<layer number="38" name="bTest" color="7" fill="1" visible="no" active="no"/>
 <layer number="39" name="tKeepout" color="4" fill="11" visible="no" active="no"/>
 <layer number="40" name="bKeepout" color="1" fill="11" visible="no" active="no"/>
@@
 <layer number="44" name="Drills" color="7" fill="1" visible="no" active="no"/>
 <layer number="45" name="Holes" color="7" fill="1" visible="no" active="no"/>
-<layer number="46" name="Milling" color="3" fill="1" visible="yes" active="no"/>
-<layer number="47" name="Measures" color="7" fill="1" visible="yes" active="no"/>
-<layer number="48" name="Document" color="7" fill="1" visible="yes" active="no"/>
-<layer number="49" name="Reference" color="7" fill="1" visible="yes" active="no"/>
-<layer number="50" name="dxf" color="7" fill="1" visible="yes" active="no"/>
-<layer number="51" name="tDocu" color="7" fill="1" visible="yes" active="no"/>
-<layer number="52" name="bDocu" color="7" fill="1" visible="yes" active="no"/>
-<layer number="53" name="tGND_GNDA" color="7" fill="9" visible="yes" active="no"/>
-<layer number="54" name="bGND_GNDA" color="1" fill="9" visible="yes" active="no"/>
-<layer number="56" name="wert" color="7" fill="1" visible="yes" active="no"/>
+<layer number="46" name="Milling" color="3" fill="1" visible="no" active="no"/>
+<layer number="47" name="Measures" color="7" fill="1" visible="no" active="no"/>
+<layer number="48" name="Document" color="7" fill="1" visible="no" active="no"/>
+<layer number="49" name="Reference" color="7" fill="1" visible="no" active="no"/>
+<layer number="50" name="dxf" color="7" fill="1" visible="no" active="no"/>
+<layer number="51" name="tDocu" color="7" fill="1" visible="no" active="no"/>
+<layer number="52" name="bDocu" color="7" fill="1" visible="no" active="no"/>
+<layer number="53" name="tGND_GNDA" color="7" fill="9" visible="no" active="no"/>
+<layer number="54" name="bGND_GNDA" color="1" fill="9" visible="no" active="no"/>
+<layer number="56" name="wert" color="7" fill="1" visible="no" active="no"/>
 <layer number="90" name="Modules" color="5" fill="1" visible="yes" active="yes"/>
 <layer number="91" name="Nets" color="2" fill="1" visible="yes" active="yes"/>
@@
 <part name="GND6" library="supply1" deviceset="GND" device=""/>
 <part name="C3" library="rcl" deviceset="C-EU" device="C0603" value="1u"/>
-<part name="R3" library="rcl" deviceset="R-EU_" device="R0603" value="3.3k"/>
-<part name="C2" library="rcl" deviceset="C-EU" device="C0603" value="10n"/>
+<part name="R3" library="rcl" deviceset="R-EU_" device="R0603" value="33k"/>
+<part name="C2" library="rcl" deviceset="C-EU" device="C0603" value="470"/>
 <part name="GND4" library="supply1" deviceset="GND" device=""/>
 <part name="R1" library="rcl" deviceset="R-EU_" device="R0603" value="22k"/>

Commit message: - ?????????? ??????
Connections:
- net N$16 renamed AINB+
- net N$17 renamed AINA+
Changed lines of the file:
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@@
 </segment>
 </net>
-<net name="N$16" class="0">
+<net name="AINB+" class="0">
 <segment>
 <pinref part="IC4" gate="G$1" pin="AINB+"/>
@@
 </segment>
 </net>
-<net name="N$17" class="0">
+<net name="AINA+" class="0">
 <segment>
 <pinref part="IC4" gate="G$1" pin="AINA+"/>

Commit message: - ???????? ???????????? ADC_DSP.sch
Parts:
- removed C21, C23, C25: 10u, rcl:C-EUC0805
- removed IC2: AD8605, analog-devices:AD8603UJ
- added SPI: (no value), con-phoenix-254:MPT4
- C1: value 10u -> 33uF; device rcl:C-EUC0805 -> rcl:CPOL-EU153CLV-0605
- C10, C6: value 1u -> 2.2u
- C13: value 1u -> 0.1u
- C5: value 1u -> 220uF; device rcl:C-EUC0603 -> rcl:CPOL-EU153CLV-0605
- C8: value 1u -> 33uF; device rcl:C-EUC0603 -> rcl:CPOL-EU153CLV-0605
- R1: value 22k -> 56
- R2: value 4.7k -> 56
- R3: value 33k -> 22k
- R4, R5: value 47k -> 33
- R6: value 1k -> 33
- R7: value 10 -> 33
Connections:
- new net N$16: C3.2, X3-1.1
- new net N$17: IC4.XTO, R1.2
- net +3V3: now also C5.+; no longer C1.1
- net +5V: no longer IC2.+VS, R4.1
- net AGND: now also C1.-, C8.-; no longer C21.2, C23.2, C25.2
- net AVCC: now also C8.+; no longer C25.1
- net GND: now also C4.2, C5.-; no longer C1.2, C5.2, C8.2, IC2.-VS, R2.2, R5.2, R6.2
- net N$1: no longer C8.1
- net N$12: now also C1.+; no longer C21.1, C23.1
- net N$19: now also IC3OSC.OSC_OUT, R2.1; no longer C4.1, IC2.IN-, IC2.OUT
- net N$2: no longer C5.1
- net N$20: now also R4.2, SPI-1.1; no longer C4.2, R6.1, R7.1
- net N$21: now also R5.2, SPI-2.1; no longer R7.2, X3-1.1
- net N$22: now also R6.2, SPI-3.1; no longer C3.2, IC2.IN+, R4.2, R5.1
- net N$23: now also C3.1; no longer R1.2
- net N$24: now also R7.2, SPI-4.1; no longer C3.1, R1.1, R2.1
- net N$3: now also C4.1
- net N$6: now also R2.2; no longer IC3OSC.OSC_OUT
- net N$8: now also R1.1; no longer IC4.XTO
- net SPI2_MISO: now also R6.1
- net SPI2_MOSI: now also R7.1
- net SPI2_NSS: now also R4.1
- net SPI2_SCK: now also R5.1
Other:
- moved on the sheet: C13, C3, C4, R1, R2, R4, R5, R6, R7, X3-1, X3-2

Commit message: - ?????? ?????????? ? ?????????????? ??????????????????
Connections:
- net +3V3: now also IC3PORTA_H.PA12
Changed lines of the file:
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@@
 <part name="R6" library="rcl" deviceset="R-EU_" device="R0603" value="33"/>
 <part name="R7" library="rcl" deviceset="R-EU_" device="R0603" value="33"/>
+<part name="+3V1" library="supply1" deviceset="+3V3" device=""/>
 </parts>
 <sheets>
@@
 <instance part="R6" gate="G$1" x="-22.86" y="0"/>
 <instance part="R7" gate="G$1" x="-27.94" y="-5.08"/>
+<instance part="+3V1" gate="G$1" x="15.24" y="45.72"/>
 </instances>
 <busses>
@@
 <junction x="114.3" y="-2.54"/>
 </segment>
+<segment>
+<pinref part="IC3" gate="PORTA_H" pin="PA12"/>
+<wire x1="25.4" y1="40.64" x2="15.24" y2="40.64" width="0.1524" layer="91"/>
+<wire x1="15.24" y1="40.64" x2="15.24" y2="43.18" width="0.1524" layer="91"/>
+<pinref part="+3V1" gate="G$1" pin="+3V3"/>
+</segment>
 </net>
